Commit message: summit_xl.urdf.xacro. Fixed wheel positions to fix movement

File: summit_xl_description/urdf/summit_xl.urdf.xacro (robot description, xacro)
@@ -139,6 +139,5 @@
     <parent link="base_link"/>
     <child link="back_right_wheel"/>
-    <!-- origin xyz="-${wheel_offset_x} -${wheel_offset_y} 0" rpy="0 0 3.1416" / -->
-    <origin xyz="-${wheel_offset_x} -${wheel_offset_y+wheel_width} 0" rpy="0 0 0" />
+    <origin xyz="-${wheel_offset_x} -${wheel_offset_y} 0" rpy="0 0 3.1416" />
     <axis xyz="0 1 0" rpy="0 0 0" />
     <limit effort="${wheel_joint_effort_limit}" velocity="${wheel_joint_velocity_limit}"/>
@@ -225,6 +224,5 @@
     <parent link="base_link"/>
     <child link="front_right_wheel"/>
-    <!-- origin xyz="${wheel_offset_x} -${wheel_offset_y} 0" rpy="0 0 3.1416" / -->
-    <origin xyz="${wheel_offset_x} -${wheel_offset_y+wheel_width} 0" rpy="0 0 0" />
+    <origin xyz="${wheel_offset_x} -${wheel_offset_y} 0" rpy="0 0 3.1416" />
     <axis xyz="0 1 0" rpy="0 0 0" />
     <limit effort="${wheel_joint_effort_limit}" velocity="${wheel_joint_velocity_limit}"/>

Commit message: Allows multiple simulations of summit xl (not omni wheels yet)

File: summit_xl_description/urdf/summit_xl.urdf.xacro (robot description, xacro)
@@ -2,5 +2,5 @@
 <robot name="summit_xl" xmlns:xacro="http://www.ros.org/wiki/xacro">
   <!-- Import all Gazebo-customization elements, including Gazebo colors -->
-  <xacro:include filename="$(find summit_xl_description)/urdf/summit_xl.gazebo" />
+  <xacro:include filename="$(find summit_xl_description)/urdf/summit_xl.gazebo"/>
   <!-- Robot mechanical and motor parameters -->
   <xacro:property name="PI" value="3.1415926535897931"/>
@@ -19,4 +19,7 @@
   <xacro:property name="ptz_joint_damping" value="0.1" />
   <xacro:property name="ptz_mechanical_reduction" value="1.0" />
+<!--
+  <xacro:property name="asd" value="$(arg namespace)"/>
+-->
   <!-- Used for fixing robot to Gazebo 'base_link' -->
   <!-- link name="world"/>
@@ -116,21 +119,21 @@
     <inertial>
       <mass value="1.250" />
-      <origin xyz="0 0 0" />
+      <origin xyz="0 0 0" rpy="0 0 ${PI}" />
       <inertia  ixx="0.0109375" ixy="0.0"  ixz="0.0"  iyy="0.021125"  iyz="0.0"  izz="0.0109375" />
     </inertial>
     <visual>
-       <origin xyz="0 0 0" rpy="0 0 0" />
-       <geometry>
-	 <mesh filename="package://summit_xl_description/meshes/summit_xl_wheel.dae" scale="1.0 1.0 1.0"/>
+       <origin xyz="0 0 0" rpy="0 0 ${PI}" />
+       <geometry>
+			   <mesh filename="package://summit_xl_description/meshes/summit_xl_wheel.dae" scale="1.0 1.0 1.0"/>
          <!-- cylinder radius="0.125" length="0.1"/ -->
        </geometry>
-	<material name="grey">
-	   <color rgba="0.5 0.5 0.5 1"/>
+	     <material name="grey">
+	       <color rgba="0.5 0.5 0.5 1"/>
        </material>
     </visual>
     <collision>
-       <origin xyz="0 0 0" rpy="0 0 0" />
-       <geometry>
-	     <mesh filename="package://summit_xl_description/meshes/summit_xl_wheel.dae" scale="1.0 1.0 1.0"/>
+       <origin xyz="0 0 0" rpy="0 0 ${PI}" />
+       <geometry>
+	       <mesh filename="package://summit_xl_description/meshes/summit_xl_wheel.dae" scale="1.0 1.0 1.0"/>
        </geometry>
     </collision>
@@ -139,5 +142,5 @@
     <parent link="base_link"/>
     <child link="back_right_wheel"/>
-    <origin xyz="-${wheel_offset_x} -${wheel_offset_y} 0" rpy="0 0 3.1416" />
+    <origin xyz="-${wheel_offset_x} -${wheel_offset_y} 0" rpy="0 0 0" />
     <axis xyz="0 1 0" rpy="0 0 0" />
     <limit effort="${wheel_joint_effort_limit}" velocity="${wheel_joint_velocity_limit}"/>
@@ -157,5 +160,5 @@
   <link name="front_left_wheel">
     <inertial>
-      <mass value="1.250" />
+      <mass value="1.250" rpy="0 0 0"/>
       <origin xyz="0 0 0" />
       <inertia  ixx="0.0109375" ixy="0.0"  ixz="0.0"  iyy="0.021125"  iyz="0.0"  izz="0.0109375" />
@@ -164,8 +167,8 @@
        <origin xyz="0 0 0" rpy="0 0 0" />
        <geometry>
-	 <mesh filename="package://summit_xl_description/meshes/summit_xl_wheel.dae" scale="1.0 1.0 1.0"/>
-       </geometry>
-	<material name="grey">
-		<color rgba="0.5 0.5 0.5 1"/>
+	       <mesh filename="package://summit_xl_description/meshes/summit_xl_wheel.dae" scale="1.0 1.0 1.0"/>
+       </geometry>
+	      <material name="grey">
+		      <color rgba="0.5 0.5 0.5 1"/>
       	</material>
     </visual>
@@ -173,5 +176,5 @@
        <origin xyz="0 0 0" rpy="0 0 0" />
        <geometry>
-	 <mesh filename="package://summit_xl_description/meshes/summit_xl_wheel.dae" scale="1.0 1.0 1.0"/>
+	       <mesh filename="package://summit_xl_description/meshes/summit_xl_wheel.dae" scale="1.0 1.0 1.0"/>
          <!-- cylinder radius="0.125" length="0.1"/ -->
        </geometry>
@@ -199,22 +202,22 @@
   <link name="front_right_wheel">
     <inertial>
-      <mass value="1.250" />
+      <mass value="1.250" rpy="0 0 ${PI}"/>
       <origin xyz="0 0 0" />
       <inertia  ixx="0.0109375" ixy="0.0"  ixz="0.0"  iyy="0.021125"  iyz="0.0"  izz="0.0109375" />
     </inertial>
     <visual>
-       <origin xyz="0 0 0" rpy="0 0 0" />
-       <geometry>
-		 <mesh filename="package://summit_xl_description/meshes/summit_xl_wheel.dae" scale="1.0 1.0 1.0"/>
+       <origin xyz="0 0 0" rpy="0 0 ${PI}" />
+       <geometry>
+		     <mesh filename="package://summit_xl_description/meshes/summit_xl_wheel.dae" scale="1.0 1.0 1.0"/>
          <!-- cylinder radius="0.125" length="0.1"/ -->
        </geometry>
-	<material name="grey">
-		<color rgba="0.5 0.5 0.5 1"/>
-      	</material>
-    </visual>
-    <collision>
-       <origin xyz="0 0 0" rpy="0 0 0" />
-       <geometry>
-	     <mesh filename="package://summit_xl_description/meshes/summit_xl_wheel.dae" scale="1.0 1.0 1.0"/>
+	     <material name="grey">
+		     <color rgba="0.5 0.5 0.5 1"/>
+       </material>
+    </visual>
+    <collision>
+       <origin xyz="0 0 0" rpy="0 0 ${PI}" />
+       <geometry>
+	       <mesh filename="package://summit_xl_description/meshes/summit_xl_wheel.dae" scale="1.0 1.0 1.0"/>
          <!-- cylinder radius="0.125" length="0.1"/ -->
        </geometry>
@@ -224,5 +227,5 @@
     <parent link="base_link"/>
     <child link="front_right_wheel"/>
-    <origin xyz="${wheel_offset_x} -${wheel_offset_y} 0" rpy="0 0 3.1416" />
+    <origin xyz="${wheel_offset_x} -${wheel_offset_y} 0" rpy="0 0 0" />
     <axis xyz="0 1 0" rpy="0 0 0" />
     <limit effort="${wheel_joint_effort_limit}" velocity="${wheel_joint_velocity_limit}"/>

File: summit_xl_description/urdf/summit_xl_fotonic.urdf.xacro (robot description, xacro)
@@ -118,22 +118,21 @@
     <inertial>
       <mass value="1.250" />
-      <origin xyz="0 0 0" />
+      <origin xyz="0 0 0" rpy="0 0 ${PI}" />
       <inertia  ixx="0.0109375" ixy="0.0"  ixz="0.0"  iyy="0.021125"  iyz="0.0"  izz="0.0109375" />
     </inertial>
     <visual>
-       <origin xyz="0 0 0" rpy="0 0 0" />
-       <geometry>
-	 <mesh filename="package://summit_xl_description/meshes/xl_fotonic/wheel.dae" scale="1.0 1.0 1.0"/>
+       <origin xyz="0 0 0" rpy="0 0 ${PI}" />
+       <geometry>
+			   <mesh filename="package://summit_xl_description/meshes/summit_xl_wheel.dae" scale="1.0 1.0 1.0"/>
          <!-- cylinder radius="0.125" length="0.1"/ -->
        </geometry>
-	<material name="grey">
-		<color rgba="0.5 0.5 0.5 1"/>
-      	</material>
-    </visual>
-    <collision>
-       <origin xyz="0 0 0" rpy="0 0 0" />
-       <geometry>
-	 <mesh filename="package://summit_xl_description/meshes/xl_fotonic/wheel.dae" scale="1.0 1.0 1.0"/>
-         <!-- cylinder radius="0.125" length="0.1"/ -->
+	     <material name="grey">
+	       <color rgba="0.5 0.5 0.5 1"/>
+       </material>
+    </visual>
+    <collision>
+       <origin xyz="0 0 0" rpy="0 0 ${PI}" />
+       <geometry>
+	       <mesh filename="package://summit_xl_description/meshes/summit_xl_wheel.dae" scale="1.0 1.0 1.0"/>
        </geometry>
     </collision>
@@ -142,5 +141,5 @@
     <parent link="base_link"/>
     <child link="back_right_wheel"/>
-    <origin xyz="-${wheel_offset_x} -${wheel_offset_y} 0" rpy="0 0 3.1416" />
+    <origin xyz="-${wheel_offset_x} -${wheel_offset_y} 0" rpy="0 0 0" />
     <axis xyz="0 1 0" rpy="0 0 0" />
     <limit effort="${wheel_joint_effort_limit}" velocity="${wheel_joint_velocity_limit}"/>
@@ -203,21 +202,23 @@
   <link name="front_right_wheel">
     <inertial>
-      <mass value="1.250" />
+      <mass value="1.250" rpy="0 0 ${PI}"/>
       <origin xyz="0 0 0" />
       <inertia  ixx="0.0109375" ixy="0.0"  ixz="0.0"  iyy="0.021125"  iyz="0.0"  izz="0.0109375" />
     </inertial>
     <visual>
-       <origin xyz="0 0 0" rpy="0 0 0" />
-       <geometry>
-	 <mesh filename="package://summit_xl_description/meshes/xl_fotonic/wheel.dae" scale="1.0 1.0 1.0"/>
-       </geometry>
-	<material name="grey">
-		<color rgba="0.5 0.5 0.5 1"/>
-      	</material>
-    </visual>
-    <collision>
-       <origin xyz="0 0 0" rpy="0 0 0" />
-       <geometry>
-	 <mesh filename="package://summit_xl_description/meshes/xl_fotonic/wheel.dae" scale="1.0 1.0 1.0"/>
+       <origin xyz="0 0 0" rpy="0 0 ${PI}" />
+       <geometry>
+		     <mesh filename="package://summit_xl_description/meshes/summit_xl_wheel.dae" scale="1.0 1.0 1.0"/>
+         <!-- cylinder radius="0.125" length="0.1"/ -->
+       </geometry>
+	     <material name="grey">
+		     <color rgba="0.5 0.5 0.5 1"/>
+       </material>
+    </visual>
+    <collision>
+       <origin xyz="0 0 0" rpy="0 0 ${PI}" />
+       <geometry>
+	       <mesh filename="package://summit_xl_description/meshes/summit_xl_wheel.dae" scale="1.0 1.0 1.0"/>
+         <!-- cylinder radius="0.125" length="0.1"/ -->
        </geometry>
     </collision>
@@ -226,5 +227,5 @@
     <parent link="base_link"/>
     <child link="front_right_wheel"/>
-    <origin xyz="${wheel_offset_x} -${wheel_offset_y} 0" rpy="0 0 3.1416" />
+    <origin xyz="${wheel_offset_x} -${wheel_offset_y} 0" rpy="0 0 0" />
     <axis xyz="0 1 0" rpy="0 0 0" />
     <limit effort="${wheel_joint_effort_limit}" velocity="${wheel_joint_velocity_limit}"/>

File: summit_xl_description/urdf/summit_xl_hq.urdf.xacro (robot description, xacro)
@@ -115,21 +115,20 @@
     <inertial>
       <mass value="1.250" />
-      <origin xyz="0 0 0" />
+      <origin xyz="0 0 0" rpy="0 0 0" />
       <inertia  ixx="0.0109375" ixy="0.0"  ixz="0.0"  iyy="0.021125"  iyz="0.0"  izz="0.0109375" />
     </inertial>
     <visual>
-       <origin xyz="0 0 0" rpy="0 0 3.1416" />
-       <!--origin xyz="0 0.075 0" rpy="0 1.57075 1.57075"/-->
-       <geometry>
-	   <mesh filename="package://summit_xl_description/meshes/high_quality/summit_xl_wheel_right.dae" scale="1.0 1.0 1.0"/>
-	   <!--cylinder radius="0.125" length="0.15"/-->
-       </geometry>
-	   <material name="grey">
-	    <color rgba="0.5 0.5 0.5 1"/>
+       <origin xyz="0 0 0" rpy="0 0 0" />
+       <geometry>
+         <mesh filename="package://summit_xl_description/meshes/high_quality/summit_xl_wheel_left.dae" scale="1.0 1.0 1.0"/>         <!-- cylinder radius="0.125" length="0.1"/ -->
+       </geometry>
+	     <material name="grey">
+	       <color rgba="0.5 0.5 0.5 1"/>
        </material>
     </visual>
     <collision>
-       <geometry>
-	    <mesh filename="package://summit_xl_description/meshes/summit_xl_wheel.dae" scale="1.0 1.0 1.0"/>
+       <origin xyz="0 0 0" rpy="0 0 0" />
+       <geometry>
+	       <mesh filename="package://summit_xl_description/meshes/summit_xl_wheel.dae" scale="1.0 1.0 1.0"/>
        </geometry>
     </collision>
@@ -138,5 +137,5 @@
     <parent link="base_link"/>
     <child link="back_right_wheel"/>
-    <origin xyz="-${wheel_offset_x} -${wheel_offset_y} 0" rpy="0 0 3.1416" />
+    <origin xyz="-${wheel_offset_x} -${wheel_offset_y} 0" rpy="0 0 0" />
     <axis xyz="0 1 0" rpy="0 0 3.1416" />
     <limit effort="${wheel_joint_effort_limit}" velocity="${wheel_joint_velocity_limit}"/>
@@ -198,22 +197,22 @@
   <link name="front_right_wheel">
     <inertial>
-      <mass value="1.250" />
+      <mass value="1.250" rpy="0 0 0"/>
       <origin xyz="0 0 0" />
       <inertia  ixx="0.0109375" ixy="0.0"  ixz="0.0"  iyy="0.021125"  iyz="0.0"  izz="0.0109375" />
     </inertial>
     <visual>
-       <origin xyz="0 0 0" rpy="0 0 3.1416" />
-       <!--origin xyz="0 0.075 0" rpy="0 1.57075 1.57075"/-->
-       <geometry>
-	   <mesh filename="package://summit_xl_description/meshes/high_quality/summit_xl_wheel_right.dae" scale="1.0 1.0 1.0"/>
-       <!--cylinder radius="0.125" length="0.15"/-->
-       </geometry>
-	   <material name="grey">
-		<color rgba="0.5 0.5 0.5 1"/>
+       <origin xyz="0 0 0" rpy="0 0 0" />
+       <geometry>
+         <mesh filename="package://summit_xl_description/meshes/high_quality/summit_xl_wheel_left.dae" scale="1.0 1.0 1.0"/>         <!-- cylinder radius="0.125" length="0.1"/ -->
+       </geometry>
+	     <material name="grey">
+		     <color rgba="0.5 0.5 0.5 1"/>
        </material>
     </visual>
     <collision>
-       <geometry>
-	    <mesh filename="package://summit_xl_description/meshes/summit_xl_wheel.dae" scale="1.0 1.0 1.0"/>
+       <origin xyz="0 0 0" rpy="0 0 0" />
+       <geometry>
+	       <mesh filename="package://summit_xl_description/meshes/summit_xl_wheel.dae" scale="1.0 1.0 1.0"/>
+         <!-- cylinder radius="0.125" length="0.1"/ -->
        </geometry>
     </collision>
@@ -222,5 +221,5 @@
     <parent link="base_link"/>
     <child link="front_right_wheel"/>
-    <origin xyz="${wheel_offset_x} -${wheel_offset_y} 0" rpy="0 0 3.1416" />
+    <origin xyz="${wheel_offset_x} -${wheel_offset_y} 0" rpy="0 0 0" />
     <axis xyz="0 1 0" rpy="0 0 3.1416" />
     <limit effort="${wheel_joint_effort_limit}" velocity="${wheel_joint_velocity_limit}"/>
