Commit message: summit_xl_description: reseting urdf files to no-multi branch

File: summit_xl_description/urdf/summit_xl.urdf.xacro (robot description, xacro)
@@ -2,5 +2,5 @@
 <robot name="summit_xl" xmlns:xacro="http://www.ros.org/wiki/xacro">
   <!-- Import all Gazebo-customization elements, including Gazebo colors -->
-  <xacro:include filename="$(find summit_xl_description)/urdf/summit_xl.gazebo"/>
+  <xacro:include filename="$(find summit_xl_description)/urdf/summit_xl.gazebo" />
   <!-- Robot mechanical and motor parameters -->
   <xacro:property name="PI" value="3.1415926535897931"/>
@@ -19,7 +19,4 @@
   <xacro:property name="ptz_joint_damping" value="0.1" />
   <xacro:property name="ptz_mechanical_reduction" value="1.0" />
-<!--
-  <xacro:property name="asd" value="$(arg namespace)"/>
--->
   <!-- Used for fixing robot to Gazebo 'base_link' -->
   <!-- link name="world"/>
@@ -119,21 +116,21 @@
     <inertial>
       <mass value="1.250" />
-      <origin xyz="0 0 0" rpy="0 0 ${PI}" />
+      <origin xyz="0 0 0" />
       <inertia  ixx="0.0109375" ixy="0.0"  ixz="0.0"  iyy="0.021125"  iyz="0.0"  izz="0.0109375" />
     </inertial>
     <visual>
-       <origin xyz="0 0 0" rpy="0 0 ${PI}" />
-       <geometry>
-			   <mesh filename="package://summit_xl_description/meshes/summit_xl_wheel.dae" scale="1.0 1.0 1.0"/>
+       <origin xyz="0 0 0" rpy="0 0 0" />
+       <geometry>
+	 <mesh filename="package://summit_xl_description/meshes/summit_xl_wheel.dae" scale="1.0 1.0 1.0"/>
          <!-- cylinder radius="0.125" length="0.1"/ -->
        </geometry>
-	     <material name="grey">
-	       <color rgba="0.5 0.5 0.5 1"/>
+	<material name="grey">
+	   <color rgba="0.5 0.5 0.5 1"/>
        </material>
     </visual>
     <collision>
-       <origin xyz="0 0 0" rpy="0 0 ${PI}" />
-       <geometry>
-	       <mesh filename="package://summit_xl_description/meshes/summit_xl_wheel.dae" scale="1.0 1.0 1.0"/>
+       <origin xyz="0 0 0" rpy="0 0 0" />
+       <geometry>
+	     <mesh filename="package://summit_xl_description/meshes/summit_xl_wheel.dae" scale="1.0 1.0 1.0"/>
        </geometry>
     </collision>
@@ -142,5 +139,6 @@
     <parent link="base_link"/>
     <child link="back_right_wheel"/>
-    <origin xyz="-${wheel_offset_x} -${wheel_offset_y} 0" rpy="0 0 0" />
+    <!-- origin xyz="-${wheel_offset_x} -${wheel_offset_y} 0" rpy="0 0 3.1416" / -->
+    <origin xyz="-${wheel_offset_x} -${wheel_offset_y+wheel_width} 0" rpy="0 0 0" />
     <axis xyz="0 1 0" rpy="0 0 0" />
     <limit effort="${wheel_joint_effort_limit}" velocity="${wheel_joint_velocity_limit}"/>
@@ -160,5 +158,5 @@
   <link name="front_left_wheel">
     <inertial>
-      <mass value="1.250" rpy="0 0 0"/>
+      <mass value="1.250" />
       <origin xyz="0 0 0" />
       <inertia  ixx="0.0109375" ixy="0.0"  ixz="0.0"  iyy="0.021125"  iyz="0.0"  izz="0.0109375" />
@@ -167,8 +165,8 @@
        <origin xyz="0 0 0" rpy="0 0 0" />
        <geometry>
-	       <mesh filename="package://summit_xl_description/meshes/summit_xl_wheel.dae" scale="1.0 1.0 1.0"/>
-       </geometry>
-	      <material name="grey">
-		      <color rgba="0.5 0.5 0.5 1"/>
+	 <mesh filename="package://summit_xl_description/meshes/summit_xl_wheel.dae" scale="1.0 1.0 1.0"/>
+       </geometry>
+	<material name="grey">
+		<color rgba="0.5 0.5 0.5 1"/>
       	</material>
     </visual>
@@ -176,5 +174,5 @@
        <origin xyz="0 0 0" rpy="0 0 0" />
        <geometry>
-	       <mesh filename="package://summit_xl_description/meshes/summit_xl_wheel.dae" scale="1.0 1.0 1.0"/>
+	 <mesh filename="package://summit_xl_description/meshes/summit_xl_wheel.dae" scale="1.0 1.0 1.0"/>
          <!-- cylinder radius="0.125" length="0.1"/ -->
        </geometry>
@@ -202,22 +200,22 @@
   <link name="front_right_wheel">
     <inertial>
-      <mass value="1.250" rpy="0 0 ${PI}"/>
+      <mass value="1.250" />
       <origin xyz="0 0 0" />
       <inertia  ixx="0.0109375" ixy="0.0"  ixz="0.0"  iyy="0.021125"  iyz="0.0"  izz="0.0109375" />
     </inertial>
     <visual>
-       <origin xyz="0 0 0" rpy="0 0 ${PI}" />
-       <geometry>
-		     <mesh filename="package://summit_xl_description/meshes/summit_xl_wheel.dae" scale="1.0 1.0 1.0"/>
+       <origin xyz="0 0 0" rpy="0 0 0" />
+       <geometry>
+		 <mesh filename="package://summit_xl_description/meshes/summit_xl_wheel.dae" scale="1.0 1.0 1.0"/>
          <!-- cylinder radius="0.125" length="0.1"/ -->
        </geometry>
-	     <material name="grey">
-		     <color rgba="0.5 0.5 0.5 1"/>
-       </material>
-    </visual>
-    <collision>
-       <origin xyz="0 0 0" rpy="0 0 ${PI}" />
-       <geometry>
-	       <mesh filename="package://summit_xl_description/meshes/summit_xl_wheel.dae" scale="1.0 1.0 1.0"/>
+	<material name="grey">
+		<color rgba="0.5 0.5 0.5 1"/>
+      	</material>
+    </visual>
+    <collision>
+       <origin xyz="0 0 0" rpy="0 0 0" />
+       <geometry>
+	     <mesh filename="package://summit_xl_description/meshes/summit_xl_wheel.dae" scale="1.0 1.0 1.0"/>
          <!-- cylinder radius="0.125" length="0.1"/ -->
        </geometry>
@@ -227,5 +225,6 @@
     <parent link="base_link"/>
     <child link="front_right_wheel"/>
-    <origin xyz="${wheel_offset_x} -${wheel_offset_y} 0" rpy="0 0 0" />
+    <!-- origin xyz="${wheel_offset_x} -${wheel_offset_y} 0" rpy="0 0 3.1416" / -->
+    <origin xyz="${wheel_offset_x} -${wheel_offset_y+wheel_width} 0" rpy="0 0 0" />
     <axis xyz="0 1 0" rpy="0 0 0" />
     <limit effort="${wheel_joint_effort_limit}" velocity="${wheel_joint_velocity_limit}"/>

File: summit_xl_description/urdf/summit_xl_fotonic.urdf.xacro (robot description, xacro)
@@ -118,21 +118,22 @@
     <inertial>
       <mass value="1.250" />
-      <origin xyz="0 0 0" rpy="0 0 ${PI}" />
+      <origin xyz="0 0 0" />
       <inertia  ixx="0.0109375" ixy="0.0"  ixz="0.0"  iyy="0.021125"  iyz="0.0"  izz="0.0109375" />
     </inertial>
     <visual>
-       <origin xyz="0 0 0" rpy="0 0 ${PI}" />
-       <geometry>
-			   <mesh filename="package://summit_xl_description/meshes/summit_xl_wheel.dae" scale="1.0 1.0 1.0"/>
+       <origin xyz="0 0 0" rpy="0 0 0" />
+       <geometry>
+	 <mesh filename="package://summit_xl_description/meshes/xl_fotonic/wheel.dae" scale="1.0 1.0 1.0"/>
          <!-- cylinder radius="0.125" length="0.1"/ -->
        </geometry>
-	     <material name="grey">
-	       <color rgba="0.5 0.5 0.5 1"/>
-       </material>
-    </visual>
-    <collision>
-       <origin xyz="0 0 0" rpy="0 0 ${PI}" />
-       <geometry>
-	       <mesh filename="package://summit_xl_description/meshes/summit_xl_wheel.dae" scale="1.0 1.0 1.0"/>
+	<material name="grey">
+		<color rgba="0.5 0.5 0.5 1"/>
+      	</material>
+    </visual>
+    <collision>
+       <origin xyz="0 0 0" rpy="0 0 0" />
+       <geometry>
+	 <mesh filename="package://summit_xl_description/meshes/xl_fotonic/wheel.dae" scale="1.0 1.0 1.0"/>
+         <!-- cylinder radius="0.125" length="0.1"/ -->
        </geometry>
     </collision>
@@ -141,5 +142,5 @@
     <parent link="base_link"/>
     <child link="back_right_wheel"/>
-    <origin xyz="-${wheel_offset_x} -${wheel_offset_y} 0" rpy="0 0 0" />
+    <origin xyz="-${wheel_offset_x} -${wheel_offset_y} 0" rpy="0 0 3.1416" />
     <axis xyz="0 1 0" rpy="0 0 0" />
     <limit effort="${wheel_joint_effort_limit}" velocity="${wheel_joint_velocity_limit}"/>
@@ -202,23 +203,21 @@
   <link name="front_right_wheel">
     <inertial>
-      <mass value="1.250" rpy="0 0 ${PI}"/>
+      <mass value="1.250" />
       <origin xyz="0 0 0" />
       <inertia  ixx="0.0109375" ixy="0.0"  ixz="0.0"  iyy="0.021125"  iyz="0.0"  izz="0.0109375" />
     </inertial>
     <visual>
-       <origin xyz="0 0 0" rpy="0 0 ${PI}" />
-       <geometry>
-		     <mesh filename="package://summit_xl_description/meshes/summit_xl_wheel.dae" scale="1.0 1.0 1.0"/>
-         <!-- cylinder radius="0.125" length="0.1"/ -->
-       </geometry>
-	     <material name="grey">
-		     <color rgba="0.5 0.5 0.5 1"/>
-       </material>
-    </visual>
-    <collision>
-       <origin xyz="0 0 0" rpy="0 0 ${PI}" />
-       <geometry>
-	       <mesh filename="package://summit_xl_description/meshes/summit_xl_wheel.dae" scale="1.0 1.0 1.0"/>
-         <!-- cylinder radius="0.125" length="0.1"/ -->
+       <origin xyz="0 0 0" rpy="0 0 0" />
+       <geometry>
+	 <mesh filename="package://summit_xl_description/meshes/xl_fotonic/wheel.dae" scale="1.0 1.0 1.0"/>
+       </geometry>
+	<material name="grey">
+		<color rgba="0.5 0.5 0.5 1"/>
+      	</material>
+    </visual>
+    <collision>
+       <origin xyz="0 0 0" rpy="0 0 0" />
+       <geometry>
+	 <mesh filename="package://summit_xl_description/meshes/xl_fotonic/wheel.dae" scale="1.0 1.0 1.0"/>
        </geometry>
     </collision>
@@ -227,5 +226,5 @@
     <parent link="base_link"/>
     <child link="front_right_wheel"/>
-    <origin xyz="${wheel_offset_x} -${wheel_offset_y} 0" rpy="0 0 0" />
+    <origin xyz="${wheel_offset_x} -${wheel_offset_y} 0" rpy="0 0 3.1416" />
     <axis xyz="0 1 0" rpy="0 0 0" />
     <limit effort="${wheel_joint_effort_limit}" velocity="${wheel_joint_velocity_limit}"/>

File: summit_xl_description/urdf/summit_xl_hq.urdf.xacro (robot description, xacro)
@@ -3,5 +3,4 @@
   <!-- Import all Gazebo-customization elements, including Gazebo colors -->
   <xacro:include filename="$(find summit_xl_description)/urdf/summit_xl_hq.gazebo" />
-  <xacro:include filename="$(find summit_xl_description)/urdf/summit_xl_base.urdf.xacro" />
   <!-- Robot mechanical and motor parameters -->
   <xacro:property name="PI" value="3.1415926535897931"/>
@@ -19,5 +18,224 @@
   <xacro:property name="ptz_joint_damping" value="0.1" />
   <xacro:property name="ptz_mechanical_reduction" value="1.0" />
-  <summit_xl_base name="summit_xl" wheels="rubber" />
+  <!-- Used for fixing robot to Gazebo 'base_link' -->
+  <!-- link name="world"/>
+  <joint name="fwf" type="planar">
+    <parent link="world"/>
+    <child link="base_footprint"/>
+  </joint -->
+  <!-- BASE FOOTPRINT -->
+  <!-- base_footprint is a fictitious link(frame) that is on the ground right below base_link origin,
+             navigation stack depends on this frame -->
+  <link name="base_footprint">
+      <visual>
+          <origin xyz="0 0 0" rpy="0 0 0" />
+          <geometry>
+             <box size="0.001 0.001 0.001" />
+          </geometry>
+      </visual>
+      <collision>
+          <origin xyz="0 0 0" rpy="0 0 0" />
+          <geometry>
+            <box size="0.001 0.001 0.001" />
+         </geometry>
+     </collision>
+  </link>
+  <joint name="base_footprint_joint" type="fixed">
+     <!-- NB While you would think this would make it go up, it is oddly reversed.
+      This moves the joint to 0,0,0 where we want it for rviz, etc. -->
+     <origin xyz="0 0 0.110" rpy="0 0 0" />
+     <parent link="base_footprint"/>
+     <child link="base_link" />
+  </joint>
+  <!-- BASE_LINK (RED) -->
+  <link name="base_link">
+    <inertial>
+      <mass value="25.0" />
+      <origin xyz="0 0 0" />
+      <inertia  ixx="1.391" ixy="0.004"  ixz="0.0"  iyy="6.853"  iyz="0.0"  izz="6.125" />
+    </inertial>
+    <visual>
+       <origin xyz="0 0 0" rpy="0 0 0" />
+       <geometry>
+	 <mesh filename="package://summit_xl_description/meshes/high_quality/summit_xl_chassis.dae"/>
+	   </geometry>
+    </visual>
+    <collision>
+       <origin xyz="0 0 0" rpy="0 0 0 " />
+       <geometry>
+         <mesh filename="package://summit_xl_description/meshes/high_quality/summit_xl_chassis.dae"/>
+	     <!-- box size = "0.750 0.4 0.3"/ -->
+       </geometry>
+    </collision>
+  </link>
+  <!-- BACK LEFT WHEEL (GREY) -->
+  <link name="back_left_wheel">
+    <inertial>
+      <mass value="1.250" />
+      <origin xyz="0 0 0"/>
+      <inertia  ixx="0.0109375" ixy="0.0"  ixz="0.0"  iyy="0.021125"  iyz="0.0"  izz="0.0109375" />
+    </inertial>
+    <visual>
+		<origin xyz="0 0 0" rpy="0 0 3.1416" />
+       <!--origin xyz="0 0.075 0" rpy="0 1.57075 1.57075"/-->
+       <geometry>
+	   <mesh filename="package://summit_xl_description/meshes/high_quality/summit_xl_wheel_left.dae" scale="1.0 1.0 1.0"/>
+		 <!--cylinder radius="0.125" length="0.15"/-->
+       </geometry>
+	<material name="grey">
+	   <color rgba="0.5 0.5 0.5 1"/>
+       </material>
+    </visual>
+    <collision>
+       <geometry>
+	    <mesh filename="package://summit_xl_description/meshes/summit_xl_wheel.dae" scale="1.0 1.0 1.0"/>
+       </geometry>
+    </collision>
+  </link>
+  <joint name="joint_back_left_wheel" type="continuous">
+    <parent link="base_link"/>
+    <child link="back_left_wheel"/>
+    <origin xyz="-${wheel_offset_x} ${wheel_offset_y} 0" rpy="0 0 0" />
+    <axis xyz="0 1 0" rpy="0 0 0" />
+    <limit effort="${wheel_joint_effort_limit}" velocity="${wheel_joint_velocity_limit}"/>
+    <joint_properties damping="${wheel_joint_damping}" friction="{wheel_joint_friction}"/>
+  </joint>
+  <transmission name="joint_blw_trans">
+	 <type>transmission_interface/SimpleTransmission</type>
+     <joint name="joint_back_left_wheel" />
+     <actuator name="joint_blw_motor">
+	    <hardwareInterface>EffortJointInterface</hardwareInterface>
+		<!-- hardwareInterface>VelocityJointInterface</hardwareInterface -->
+        <mechanicalReduction>${wheel_mechanical_reduction}</mechanicalReduction>
+     	<!-- motorTorqueConstant>1</motorTorqueConstant -->
+     </actuator>
+  </transmission>
+  <!-- BACK RIGHT WHEEL (GREY) -->
+  <link name="back_right_wheel">
+    <inertial>
+      <mass value="1.250" />
+      <origin xyz="0 0 0" />
+      <inertia  ixx="0.0109375" ixy="0.0"  ixz="0.0"  iyy="0.021125"  iyz="0.0"  izz="0.0109375" />
+    </inertial>
+    <visual>
+       <origin xyz="0 0 0" rpy="0 0 3.1416" />
+       <!--origin xyz="0 0.075 0" rpy="0 1.57075 1.57075"/-->
+       <geometry>
+	   <mesh filename="package://summit_xl_description/meshes/high_quality/summit_xl_wheel_right.dae" scale="1.0 1.0 1.0"/>
+	   <!--cylinder radius="0.125" length="0.15"/-->
+       </geometry>
+	   <material name="grey">
+	    <color rgba="0.5 0.5 0.5 1"/>
+       </material>
+    </visual>
+    <collision>
+       <geometry>
+	    <mesh filename="package://summit_xl_description/meshes/summit_xl_wheel.dae" scale="1.0 1.0 1.0"/>
+       </geometry>
+    </collision>
+  </link>
+  <joint name="joint_back_right_wheel" type="continuous">
+    <parent link="base_link"/>
+    <child link="back_right_wheel"/>
+    <origin xyz="-${wheel_offset_x} -${wheel_offset_y} 0" rpy="0 0 3.1416" />
+    <axis xyz="0 1 0" rpy="0 0 3.1416" />
+    <limit effort="${wheel_joint_effort_limit}" velocity="${wheel_joint_velocity_limit}"/>
+    <joint_properties damping="${wheel_joint_damping}" friction="{wheel_joint_friction}"/>
+  </joint>
+  <transmission name="joint_brw_trans">
+    <type>transmission_interface/SimpleTransmission</type>
+    <joint name="joint_back_right_wheel" />
+    <actuator name="joint_brw_motor">
+	   <hardwareInterface>EffortJointInterface</hardwareInterface>
+       <!-- hardwareInterface>VelocityJointInterface</hardwareInterface -->
+       <mechanicalReduction>${wheel_mechanical_reduction}</mechanicalReduction>
+	   <!-- motorTorqueConstant>1</motorTorqueConstant -->
+    </actuator>
+  </transmission>
+  <!-- FRONT LEFT WHEEL (GREY) -->
+  <link name="front_left_wheel">
+    <inertial>
+      <mass value="1.250" />
+      <origin xyz="0 0 0" />
+      <inertia  ixx="0.0109375" ixy="0.0"  ixz="0.0"  iyy="0.021125"  iyz="0.0"  izz="0.0109375" />
+    </inertial>
+    <visual>
+      <origin xyz="0 0 0" rpy="0 0 3.1416" />
+      <!--origin xyz="0 0.075 0" rpy="0 1.57075 1.57075"/-->
+      <geometry>
+	  <mesh filename="package://summit_xl_description/meshes/high_quality/summit_xl_wheel_left.dae" scale="1.0 1.0 1.0"/>
+	  <!--cylinder radius="0.125" length="0.15"/-->
+      </geometry>
+	  <material name="grey">
+	    <color rgba="0.5 0.5 0.5 1"/>
+      </material>
+    </visual>
+    <collision>
+       <geometry>
+	    <mesh filename="package://summit_xl_description/meshes/summit_xl_wheel.dae" scale="1.0 1.0 1.0"/>
+       </geometry>
+    </collision>
+  </link>
+  <joint name="joint_front_left_wheel" type="continuous">
+    <parent link="base_link"/>
+    <child link="front_left_wheel"/>
+    <origin xyz="${wheel_offset_x} ${wheel_offset_y} 0" rpy="0 0 0" />
+    <axis xyz="0 1 0" rpy="0 0 0" />
+    <limit effort="${wheel_joint_effort_limit}" velocity="${wheel_joint_velocity_limit}"/>
+    <joint_properties damping="${wheel_joint_damping}" friction="{wheel_joint_friction}"/>
+  </joint>
+  <transmission name="joint_flw_trans">
+	 <type>transmission_interface/SimpleTransmission</type>
+     <joint name="joint_front_left_wheel" />
+     <actuator name="joint_flw_motor">
+	   <hardwareInterface>EffortJointInterface</hardwareInterface>
+       <!-- hardwareInterface>VelocityJointInterface</hardwareInterface -->
+       <mechanicalReduction>${wheel_mechanical_reduction}</mechanicalReduction>
+       <!-- motorTorqueConstant>1</motorTorqueConstant -->
+     </actuator>
+  </transmission>
+  <!-- FRONT RIGHT WHEEL (GREY) -->
+  <link name="front_right_wheel">
+    <inertial>
+      <mass value="1.250" />
+      <origin xyz="0 0 0" />
+      <inertia  ixx="0.0109375" ixy="0.0"  ixz="0.0"  iyy="0.021125"  iyz="0.0"  izz="0.0109375" />
+    </inertial>
+    <visual>
+       <origin xyz="0 0 0" rpy="0 0 3.1416" />
+       <!--origin xyz="0 0.075 0" rpy="0 1.57075 1.57075"/-->
+       <geometry>
+	   <mesh filename="package://summit_xl_description/meshes/high_quality/summit_xl_wheel_right.dae" scale="1.0 1.0 1.0"/>
+       <!--cylinder radius="0.125" length="0.15"/-->
+       </geometry>
+	   <material name="grey">
+		<color rgba="0.5 0.5 0.5 1"/>
+       </material>
+    </visual>
+    <collision>
+       <geometry>
+	    <mesh filename="package://summit_xl_description/meshes/summit_xl_wheel.dae" scale="1.0 1.0 1.0"/>
+       </geometry>
+    </collision>
+  </link>
+  <joint name="joint_front_right_wheel" type="continuous">
+    <parent link="base_link"/>
+    <child link="front_right_wheel"/>
+    <origin xyz="${wheel_offset_x} -${wheel_offset_y} 0" rpy="0 0 3.1416" />
+    <axis xyz="0 1 0" rpy="0 0 3.1416" />
+    <limit effort="${wheel_joint_effort_limit}" velocity="${wheel_joint_velocity_limit}"/>
+    <joint_properties damping="${wheel_joint_damping}" friction="{wheel_joint_friction}"/>
+  </joint>
+  <transmission name="joint_frw_trans">
+	 <type>transmission_interface/SimpleTransmission</type>
+     <joint name="joint_front_right_wheel" />
+     <actuator name="joint_frw_motor">
+	   <hardwareInterface>EffortJointInterface</hardwareInterface>
+	   <!-- hardwareInterface>VelocityJointInterface</hardwareInterface -->
+       <mechanicalReduction>${wheel_mechanical_reduction}</mechanicalReduction>
+       <!-- motorTorqueConstant>1</motorTorqueConstant -->
+     </actuator>
+     <!-- motorTorqueConstant>1</motorTorqueConstant -->
+  </transmission>
   <!-- HOKUYO SENSOR -->
   <joint name="hokuyo_laser_joint" type="fixed">
