Commit message: summit_xl_description: fixing rubber_wheel bug

File: summit_xl_description/urdf/wheels/rubber_wheel.urdf.xacro (robot description, xacro)
@@ -88,5 +88,5 @@
       </actuator>
     </transmission>
-        <gazebo reference="${name}_wheel">
+    <gazebo reference="${name}_wheel">
 			<mu1 value="5.0"/>
 			<mu2 value="0.5"/>
@@ -98,5 +98,5 @@
     </gazebo>
     <gazebo reference="cover_${name}1_wheel">
-      <material>Gazebo/Gray</material>
+      <material>Gazebo/Grey</material>
     </gazebo>
   </xacro:macro>
