Commit message: summit_xl_description: moving axis mesh to sensors folder

File: summit_xl_description/urdf/sensors/axis.urdf.xacro (robot description, xacro)
@@ -29,5 +29,5 @@
         </material>
 	      <geometry>
-					<mesh filename= "package://summit_xl_description/meshes/xl_fotonic/axis_p5512.stl" scale="1.0 1.0 1.0"/>
+					<mesh filename= "package://summit_xl_description/meshes/sensors/axis_p5512.stl" scale="1.0 1.0 1.0"/>
 	      </geometry>
 	    </visual>
@@ -35,5 +35,5 @@
 	      <origin xyz="0.03 0.0 -0.3" rpy="0 0 0"/>
 	      <geometry>
-	        <mesh filename= "package://summit_xl_description/meshes/xl_fotonic/axis_p5512.stl" scale="1.0 1.0 1.0"/>
+	        <mesh filename= "package://summit_xl_description/meshes/sensors/axis_p5512.stl" scale="1.0 1.0 1.0"/>
 	      </geometry>
 	    </collision>
