Commit message: gps sensor description. Bug fixed.

File: summit_xl_description/urdf/sensors/gps.urdf.xacro (robot description, xacro)
@@ -9,5 +9,5 @@
 	    <child link="${name}_link"/>
 	  </joint>
-	  <link name="gps_link">
+	  <link name="${name}_link">
 	    <inertial>
 	      <mass value="0.001"/>
