Commit message: summit_xl_description: summit_x, adding gazebo and rviz colors

File: summit_xl_description/urdf/bases/summit_x_base.gazebo.xacro (robot description, xacro)
@@ -51,9 +51,6 @@
     <material>Gazebo/Grey</material>
   </gazebo>
-  <gazebo reference="logos_link">
-    <material>Gazebo/Red</material>
-  </gazebo>
-  <gazebo reference="covers_link">
-    <material>Gazebo/Grey</material>
+  <gazebo reference="rover_link">
+    <material>Gazebo/FlatBlack</material>
   </gazebo>
 </robot>

File: summit_xl_description/urdf/bases/summit_x_base.urdf.xacro (robot description, xacro)
@@ -38,7 +38,32 @@
 			<origin xyz="0 0 0" rpy="0 0 0" />
 			<geometry>
-				<mesh filename="package://summit_xl_description/meshes/x_wam/chassis_xwam_down.dae"/>
+				<mesh filename="package://summit_xl_description/meshes/x_wam/chassis_xwam_down.stl"/>
 			</geometry>
-			<material name="darkgrey">
+			<material name="summit_x_base_color">
+				<color rgba="0.6 0.6 0.6 1"/>
+			</material>
+		</visual>
+		<collision>
+			<origin xyz="0 0 0" rpy="0 0 0 " />
+				<geometry>
+					<mesh filename="package://summit_xl_description/meshes/x_wam/chassis_xwam_down.stl"/>
+				</geometry>
+		</collision>
+	</link>
+	<!-- ***************************** -->
+  <!-- ROVER PART - UP SCISSOR MECH  -->
+  <!-- ***************************** -->
+	<link name="rover_link">
+		<inertial>
+			<mass value="1.0" /> <!-- 20.0 -->
+			<origin xyz="0 0 0" />
+			<inertia  ixx="0.2185" ixy="0.0"  ixz="-0.001"  iyy="0.33677"  iyz="0.0"  izz="0.20511" />
+		</inertial>
+		<visual>
+			<origin xyz="0 0 0" rpy="0 0 0" />
+			<geometry>
+				<mesh filename="package://summit_xl_description/meshes/x_wam/chassis_xwam_up.stl"/>
+			</geometry>
+			<material name="summit_x_rover_color">
 				<color rgba="0.1 0.1 0.1 1"/>
 			</material>
@@ -46,31 +71,9 @@
 		<collision>
 			<origin xyz="0 0 0" rpy="0 0 0 " />
-				<geometry>
-					<mesh filename="package://summit_xl_description/meshes/x_wam/chassis_xwam_down.dae"/>
-				</geometry>
+			<geometry>
+				<mesh filename="package://summit_xl_description/meshes/x_wam/chassis_xwam_up.stl"/>
+			</geometry>
 		</collision>
 	</link>
-	  <!-- ***************************** -->
-  <!-- ROVER PART - UP SCISSOR MECH  -->
-  <!-- ***************************** -->
-  <link name="rover_link">
-    <inertial>
-      <mass value="1.0" /> <!-- 20.0 -->
-      <origin xyz="0 0 0" />
-      <inertia  ixx="0.2185" ixy="0.0"  ixz="-0.001"  iyy="0.33677"  iyz="0.0"  izz="0.20511" />
-    </inertial>
-    <visual>
-       <origin xyz="0 0 0" rpy="0 0 0" />
-       <geometry>
-	   <mesh filename="package://summit_xl_description/meshes/x_wam/chassis_xwam_up.dae"/>
-       </geometry>
-    </visual>
-    <collision>
-       <origin xyz="0 0 0" rpy="0 0 0 " />
-       <geometry>
-       <mesh filename="package://summit_xl_description/meshes/x_wam/chassis_xwam_up.dae"/>
-       </geometry>
-    </collision>
-  </link>
   <joint name="scissor_prismatic_joint" type="prismatic">
     <parent link="base_link"/>

Commit message: summit_xl_description: adding axis sensor to summit X chasis

File: summit_xl_description/urdf/bases/summit_x_base.gazebo.xacro (robot description, xacro)
@@ -54,3 +54,39 @@
     <material>Gazebo/FlatBlack</material>
   </gazebo>
+  <gazebo reference="camera_tilt_link">
+    <sensor type="camera" name="camera1">
+      <update_rate>30.0</update_rate>
+      <camera name="head">
+        <horizontal_fov>1.3962634</horizontal_fov>
+        <image>
+          <width>800</width>
+          <height>800</height>
+          <format>R8G8B8</format>
+        </image>
+        <clip>
+          <near>0.03</near>
+          <far>300</far>
+        </clip>
+        <noise>
+          <type>gaussian</type>
+          <mean>0.0</mean>
+          <stddev>0.007</stddev>
+        </noise>
+      </camera>
+      <plugin name="camera_controller" filename="libgazebo_ros_camera.so">
+        <alwaysOn>true</alwaysOn>
+        <updateRate>0.0</updateRate>
+        <cameraName>camera</cameraName>
+        <imageTopicName>image_raw</imageTopicName>
+        <cameraInfoTopicName>camera_info</cameraInfoTopicName>
+        <frameName>camera_tilt_link</frameName>
+        <hackBaseline>0.07</hackBaseline>
+        <distortionK1>0.0</distortionK1>
+        <distortionK2>0.0</distortionK2>
+        <distortionK3>0.0</distortionK3>
+        <distortionT1>0.0</distortionT1>
+        <distortionT2>0.0</distortionT2>
+      </plugin>
+    </sensor>
+  </gazebo>
 </robot>

File: summit_xl_description/urdf/bases/summit_x_base.urdf.xacro (robot description, xacro)
@@ -91,38 +91,70 @@
 	 </actuator>
   </transmission>
-  <!-- ***************************** -->
-  <!-- SCISSOR MECHANISM PART 1      -->
-  <!-- ***************************** -->
-<!--
-  <joint name="scissor_bars1_joint" type="continuous">
-    <parent link="rover_link"/>
-    <child link="scissor_bars1_link"/>
-    <origin xyz="0 0 0" rpy="0.0 0.0 0.0"/>
-    <limit effort="300" velocity="10.0" lower="-20.2" upper="20.7" />
-    <mimic joint="scissor_prismatic_joint" multiplier="5" offset="0.0" />
-    <axis xyz="0 1 0" />
+	<!-- Axis camera -->
+	<xacro:property name="ptz_joint_effort_limit" value="100.0" />
+  <xacro:property name="ptz_joint_velocity_limit" value="100.0"/>
+  <xacro:property name="ptz_joint_friction" value="0.1" />
+  <xacro:property name="ptz_joint_damping" value="0.1" />
+  <xacro:property name="ptz_mechanical_reduction" value="1.0" />
+	<joint name="camera_joint" type="fixed">
+			<axis xyz="0 1 0" />
+			<origin xyz="0.0 0.0 0.13" rpy="0.0 ${PI/4} 0.0"/>
+      <parent link="rover_link"/>
+      <child link="camera_link"/>
   </joint>
-	<link name="scissor_bars1_link">
-    <inertial>
-      <mass value="1" />
-      <origin xyz="0 0 0" rpy="0 -3.1415 0"/>
-			<box_inertia m="1" x="0.5" y="0.2" z="0.05"/>
+	<link name="camera_link">
+		<inertial>
+			<origin xyz="0.03 0.0 -0.3" rpy="0 0 0"/>
+			<mass value="0.1" />
+			<origin xyz="0 0 0" rpy="0 0 0" />
+			<inertia ixx="0.1" ixy="0" ixz="0" iyy="0.1" iyz="0" izz="0.1" />
+		</inertial>
+	</link>
+  <joint name="joint_camera_pan" type="continuous">
+     <axis xyz="0 0 1" />
+     <origin xyz="0.0 0.0 0.1"/>
+     <parent link="camera_link"/>
+     <child link="camera_pan_link"/>
+     <limit effort="${ptz_joint_effort_limit}" velocity="${ptz_joint_velocity_limit}" lower="-3.1416" upper="3.1416"/>
+     <joint_properties damping="${ptz_joint_damping}" friction="{ptz_joint_friction}"/>
+  </joint>
+  <link name="camera_pan_link">
+     <inertial>
+       <mass value="0.1" />
+       <origin xyz="0 0 0" rpy="0 0 0" />
+       <inertia ixx="0.1" ixy="0" ixz="0" iyy="0.1" iyz="0" izz="0.1" />
     </inertial>
-    <visual>
-       <origin xyz="0 0 0" rpy="0 -3.1415 0" />
-       <geometry>
-					<mesh filename="package://summit_xl_description/meshes/x_wam/scissor_bars_1.stl"/>
-					<box x="0.2" y="0.1" z="0.1"/>
-       </geometry>
-    </visual>
-    <collision>
-       <origin xyz="0 0 0" rpy="0 -3.1415 0" />
-       <geometry>
-				<mesh filename="package://summit_xl_description/meshes/x_wam/scissor_bars_1.stl"/>
-				<box x="0.2" y="0.1" z="0.1"/>
-       </geometry>
-    </collision>
   </link>
--->
+  <transmission name="camera_pan_trans">
+	 <type>transmission_interface/SimpleTransmission</type>
+     <joint name="joint_camera_pan" />
+     <actuator name="pan_motor">
+		   <hardwareInterface>EffortJointInterface</hardwareInterface>
+       <mechanicalReduction>${ptz_mechanical_reduction}</mechanicalReduction>
+     </actuator>
+  </transmission>
+  <joint name="joint_camera_tilt" type="continuous">
+     <axis xyz="0 1 0" />
+     <origin xyz="0.0 0.0 0.0"/>
+     <parent link="camera_pan_link"/>
+     <child link="camera_tilt_link"/>
+     <limit effort="${ptz_joint_effort_limit}" velocity="${ptz_joint_velocity_limit}" lower="-1.5708" upper="1.5708"/>
+     <joint_properties damping="${ptz_joint_damping}" friction="{ptz_joint_friction}"/>
+  </joint>
+  <link name="camera_tilt_link">
+     <inertial>
+       <mass value="0.1" />
+       <origin xyz="0 0 0" rpy="0 0 0" />
+       <inertia ixx="0.1" ixy="0" ixz="0" iyy="0.1" iyz="0" izz="0.1" />
+    </inertial>
+  </link>
+  <transmission name="camera_tilt_trans">
+	 <type>transmission_interface/SimpleTransmission</type>
+     <joint name="joint_camera_tilt" />
+     <actuator name="tilt_motor">
+			 <hardwareInterface>EffortJointInterface</hardwareInterface>
+			 <mechanicalReduction>${ptz_mechanical_reduction}</mechanicalReduction>
+     </actuator>
+  </transmission>
 	</xacro:macro>
 </robot>

Commit message: summit_xl_description: adding hokuyo sensor to Summit X chassis

File: summit_xl_description/urdf/bases/summit_x_base.gazebo.xacro (robot description, xacro)
@@ -90,3 +90,34 @@
     </sensor>
   </gazebo>
+  <gazebo reference="hokuyo_laser_link">
+		<sensor type="ray" name="hokuyo_sensor">
+			<pose>0 0 0 0 0 0</pose>
+			<visualize>false</visualize>
+			<update_rate>30</update_rate>
+			<ray>
+				<scan>
+					<horizontal>
+						<samples>1081</samples>
+						<resolution>1</resolution>
+						<min_angle>2.35619449</min_angle>  <!-- +/-135 deg -->
+						<max_angle>-2.35619449</max_angle>
+					</horizontal>
+				</scan>
+				<range>
+					<min>0.10</min>
+					<max>30.0</max>
+					<resolution>0.01</resolution>
+				</range>
+				<noise>
+					<type>gaussian</type>
+					<mean>0.0</mean>
+					<stddev>0.01</stddev>
+				</noise>
+			</ray>
+			<plugin name="gazebo_ros_head_hokuyo_controller" filename="libgazebo_ros_laser.so">
+				<topicName>hokuyo/scan</topicName>
+				<frameName>hokuyo_laser_link</frameName>
+			</plugin>
+		</sensor>
+	</gazebo>
 </robot>

File: summit_xl_description/urdf/bases/summit_x_base.urdf.xacro (robot description, xacro)
@@ -157,4 +157,17 @@
      </actuator>
   </transmission>
+	<!-- Hokuyo sensor -->
+	<joint name="hokuyo_laser_joint" type="fixed">
+		<origin xyz="0.075 0.0 0.0" rpy="${PI} 0 0"/>
+		<parent link="rover_link"/>
+		<child link="hokuyo_laser_link"/>
+	</joint>
+	<link name="hokuyo_laser_link">
+		<inertial>
+			<mass value="1e-5" />
+			<origin xyz="0 0 0" rpy="0 0 0"/>
+			<inertia ixx="1e-6" ixy="0" ixz="0" iyy="1e-6" iyz="0" izz="1e-6" />
+		</inertial>
+	</link>
 	</xacro:macro>
 </robot>

File: summit_xl_description/urdf/sensors/hokuyo_utm30lx.urdf.xacro (robot description, xacro)
@@ -64,5 +64,5 @@
 				</plugin>
 			</sensor>
-	</gazebo>
+		</gazebo>
   </xacro:macro>
 </robot>
