Commit message: summit_xl_description: switching to .dae model

File: summit_xl_description/urdf/bases/summit_xl_base.gazebo.xacro (robot description, xacro)
@@ -48,4 +48,5 @@
     <material>Gazebo/Green</material>
   </gazebo>
+<!--
   <gazebo reference="base_link">
     <material>Gazebo/Black</material>
@@ -57,3 +58,4 @@
     <material>Gazebo/Grey</material>
   </gazebo>
+-->
 </robot>

File: summit_xl_description/urdf/bases/summit_xl_base.urdf.xacro (robot description, xacro)
@@ -41,5 +41,5 @@
        <xacro:if value="${hq}">
        <geometry>
-	     <mesh filename="package://summit_xl_description/meshes/bases/summit_xl_chassis.stl"/>
+	     <mesh filename="package://summit_xl_description/meshes/bases/summit_xl_chassis.dae"/>
        </geometry>
        </xacro:if>
@@ -61,4 +61,5 @@
   </link>
   <!-- COVERS AND SUSPENSIONS -->
+<!--
   <xacro:if value="${hq}">
   <joint name="covers_joint" type="fixed">
@@ -79,5 +80,7 @@
   </link>
   </xacro:if>
+-->
   <!-- LOGOS -->
+<!--
   <joint name="logos_joint" type="fixed">
      <origin xyz="0 0 0" rpy="0 0 0" />
@@ -85,9 +88,11 @@
      <child link="logos_link" />
   </joint>
+-->
+<!--
   <link name="logos_link">
     <visual>
        <origin xyz="0 0 0" rpy="0 0 0" />
        <geometry>
-	     <mesh filename="package://summit_xl_description/meshes/bases/summit_xl_logos.stl" scale="1.001 1.001 1.001"/> <!-- Scaled a little bit up to avoid visualization problems -->
+	     <mesh filename="package://summit_xl_description/meshes/bases/summit_xl_logos.stl" scale="1.001 1.001 1.001"/>
        </geometry>
        <material name="red">
@@ -96,4 +101,5 @@
     </visual>
   </link>
+-->
   </xacro:macro>
 </robot>

File: summit_xl_description/urdf/wheels/rubber_wheel.urdf.xacro (robot description, xacro)
@@ -27,5 +27,5 @@
           <origin xyz="0 0 0" rpy="0 0 0" />
           <geometry>
-            <mesh filename="package://summit_xl_description/meshes/wheels/rubber_wheel.stl" />
+            <mesh filename="package://summit_xl_description/meshes/wheels/rubber_wheel.dae" />
           </geometry>
         </xacro:if>
@@ -37,7 +37,9 @@
           </geometry>
         </xacro:unless>
+<!--
         <material name="darkgrey">
            <color rgba="0.2 0.2 0.2 1"/>
         </material>
+-->
       </visual>
       <collision>
@@ -63,9 +65,11 @@
 		<origin xyz="0 0 0" rpy="${reflect*PI} 0 0" />
         <geometry>
-          <mesh filename="package://summit_xl_description/meshes/wheels/rubber_wheel_cover.stl" />
+          <mesh filename="package://summit_xl_description/meshes/wheels/rubber_wheel_cover.dae" />
         </geometry>
+<!--
         <material name="lightgrey">
            <color rgba="0.6 0.6 0.6 1"/>
         </material>
+-->
       </visual>
 <!-- MOTOR VISUAL -->
