Commit message: Kinect instance in summi_xl_hq.urdf

File: summit_xl_description/robots/summit_xl_hq.urdf.xacro (robot description, xacro)
@@ -5,4 +5,5 @@
   <xacro:include filename="$(find summit_xl_description)/urdf/bases/summit_xl_base.urdf.xacro" />
     <xacro:include filename="$(find summit_xl_description)/urdf/wheels/rubber_wheel.urdf.xacro" />
+    <xacro:include filename="$(find summit_xl_description)/urdf/sensors/kinect.urdf.xacro" />
   <!-- Robot mechanical and motor parameters -->
   <xacro:property name="PI" value="3.1415926535897931"/>
@@ -61,3 +62,6 @@
       </collision>
   </link>
+  <sensor_kinect name="kinect1" parent="base_link">
+    <origin xyz="0.33 0 0.33" rpy="0 0 0"/>
+  </sensor_kinect>
 </robot>

Commit message: New wheels added.

File: summit_xl_description/robots/summit_xl_hq.urdf.xacro (robot description, xacro)
@@ -4,6 +4,6 @@
   <xacro:include filename="$(find summit_xl_description)/urdf/summit_xl_hq.gazebo" />
   <xacro:include filename="$(find summit_xl_description)/urdf/bases/summit_xl_base.urdf.xacro" />
-    <xacro:include filename="$(find summit_xl_description)/urdf/wheels/rubber_wheel.urdf.xacro" />
-    <xacro:include filename="$(find summit_xl_description)/urdf/sensors/kinect.urdf.xacro" />
+  <xacro:include filename="$(find summit_xl_description)/urdf/wheels/rubber_wheel.urdf.xacro" />
+  <xacro:include filename="$(find summit_xl_description)/urdf/sensors/kinect.urdf.xacro" />
   <!-- Robot mechanical and motor parameters -->
   <xacro:property name="PI" value="3.1415926535897931"/>

File: summit_xl_description/urdf/sensors/kinect.urdf.xacro (robot description, xacro)
@@ -2,42 +2,4 @@
 <robot name="sensor_kinect" xmlns:xacro="http://ros.org/wiki/xacro">
 	<xacro:property name="M_PI" value="3.1415926535897931" />
-	<xacro:macro name="kinect_sim_3dsensor">
-    <gazebo reference="camera_link">
-      <sensor type="depth" name="camera">
-        <always_on>true</always_on>
-        <update_rate>20.0</update_rate>
-        <camera>
-          <horizontal_fov>${60.0*M_PI/180.0}</horizontal_fov>
-          <image>
-            <format>R8G8B8</format>
-            <width>640</width>
-            <height>480</height>
-          </image>
-          <clip>
-            <near>0.05</near>
-            <far>8.0</far>
-          </clip>
-        </camera>
-        <plugin name="kinect_camera_controller" filename="libgazebo_ros_openni_kinect.so">
-          <cameraName>${name}</cameraName>
-          <alwaysOn>true</alwaysOn>
-          <updateRate>10</updateRate>
-          <imageTopicName>rgb/image_raw</imageTopicName>
-          <depthImageTopicName>depth/image_raw</depthImageTopicName>
-          <pointCloudTopicName>depth/points</pointCloudTopicName>
-          <cameraInfoTopicName>rgb/camera_info</cameraInfoTopicName>
-          <depthImageCameraInfoTopicName>depth/camera_info</depthImageCameraInfoTopicName>
-          <frameName>${name}_camera_depth_optical_frame</frameName>
-          <baseline>0.1</baseline>
-          <distortion_k1>0.0</distortion_k1>
-          <distortion_k2>0.0</distortion_k2>
-          <distortion_k3>0.0</distortion_k3>
-          <distortion_t1>0.0</distortion_t1>
-          <distortion_t2>0.0</distortion_t2>
-          <pointCloudCutoff>0.4</pointCloudCutoff>
-        </plugin>
-      </sensor>
-    </gazebo>
-  </xacro:macro>
   <!-- Parameterised in part by the values in turtlebot_properties.urdf.xacro -->
   <xacro:macro name="sensor_kinect" params="name parent *origin">
@@ -130,3 +92,41 @@
 	<kinect_sim_3dsensor/>
   </xacro:macro>
+  	<xacro:macro name="kinect_sim_3dsensor">
+    <gazebo reference="camera_link">
+      <sensor type="depth" name="camera">
+        <always_on>true</always_on>
+        <update_rate>20.0</update_rate>
+        <camera>
+          <horizontal_fov>${60.0*M_PI/180.0}</horizontal_fov>
+          <image>
+            <format>R8G8B8</format>
+            <width>640</width>
+            <height>480</height>
+          </image>
+          <clip>
+            <near>0.05</near>
+            <far>8.0</far>
+          </clip>
+        </camera>
+        <plugin name="kinect_camera_controller" filename="libgazebo_ros_openni_kinect.so">
+          <cameraName>${name}</cameraName>
+          <alwaysOn>true</alwaysOn>
+          <updateRate>10</updateRate>
+          <imageTopicName>rgb/image_raw</imageTopicName>
+          <depthImageTopicName>depth/image_raw</depthImageTopicName>
+          <pointCloudTopicName>depth/points</pointCloudTopicName>
+          <cameraInfoTopicName>rgb/camera_info</cameraInfoTopicName>
+          <depthImageCameraInfoTopicName>depth/camera_info</depthImageCameraInfoTopicName>
+          <frameName>${name}_camera_depth_optical_frame</frameName>
+          <baseline>0.1</baseline>
+          <distortion_k1>0.0</distortion_k1>
+          <distortion_k2>0.0</distortion_k2>
+          <distortion_k3>0.0</distortion_k3>
+          <distortion_t1>0.0</distortion_t1>
+          <distortion_t2>0.0</distortion_t2>
+          <pointCloudCutoff>0.4</pointCloudCutoff>
+        </plugin>
+      </sensor>
+    </gazebo>
+  </xacro:macro>
 </robot>

Commit message: Wheels OK

File: summit_xl_description/robots/summit_xl_hq.urdf.xacro (robot description, xacro)
@@ -9,5 +9,5 @@
   <xacro:property name="PI" value="3.1415926535897931"/>
   <xacro:property name="wheel_offset_x" value="0.223" />    <!-- x,y,z in base_link CS -->
-  <xacro:property name="wheel_offset_y" value="0.154" />
+  <xacro:property name="wheel_offset_y" value="0.234" />
   <xacro:property name="wheel_offset_z" value="0.0" />
   <xacro:property name="wheel_joint_damping" value="0.0" />
@@ -21,4 +21,5 @@
   <xacro:property name="ptz_joint_damping" value="0.1" />
   <xacro:property name="ptz_mechanical_reduction" value="1.0" />
+  <xacro:property name="rubber_wheels" value="true" />
   <xacro:property name="rubber_wheels" value="true" />
   <summit_xl_base name="summit_xl" />
@@ -65,3 +66,6 @@
     <origin xyz="0.33 0 0.33" rpy="0 0 0"/>
   </sensor_kinect>
+  <sensor_kinect name="kinect2" parent="base_link">
+    <origin xyz="0.33 0 0.43" rpy="0 0 0"/>
+  </sensor_kinect>
 </robot>

File: summit_xl_description/urdf/wheels/rubber_wheel.urdf.xacro (robot description, xacro)
@@ -5,7 +5,4 @@
   <property name="wheel_height" value="0.14" />
   <property name="wheel_mass" value="2.5" /> <!-- in kg-->
-  <property name="base_x_origin_to_wheel_origin" value="0.22911" />
-  <property name="base_y_origin_to_wheel_origin" value="0.23350" />
-  <property name="base_z_origin_to_wheel_origin" value="0.0" />
   <macro name="cylinder_inertia" params="m r h">
     <inertia  ixx="${m*(3*r*r+h*h)/12}" ixy = "0" ixz = "0"
@@ -14,13 +11,24 @@
   </macro>
   <xacro:macro name="rubber_wheel" params="name parent *origin reflect">
+    <joint name="joint_${name}_wheel" type="continuous">
+      <parent link="${parent}"/>
+      <child link="${name}_wheel"/>
+      <insert_block name="origin" />
+      <axis xyz="0 1 0" rpy="0 0 0" />
+      <limit effort="100" velocity="100"/>
+      <joint_properties damping="0.0" friction="0.0"/>
+    </joint>
     <link name="${name}_wheel">
       <visual>
-		<origin xyz="0 0 0" rpy="${PI*reflect} 0 0" />
+		<origin xyz="0 0 0" rpy="0 0 0" />
         <geometry>
-          <mesh filename="package://summit_xl_description/meshes/wheels/summit_xl_wheel_right.stl" />
+          <mesh filename="package://summit_xl_description/meshes/wheels/rubber_wheel.stl" />
         </geometry>
+        <material name="darkgrey">
+           <color rgba="0.2 0.2 0.2 1"/>
+        </material>
       </visual>
       <collision>
-		<origin xyz="0 0 0" rpy="0 0 ${PI*reflect}" />
+		<origin xyz="0 0 0" rpy="0 0 0" />
         <geometry>
           <cylinder length="${wheel_height}" radius="${wheel_radius}" />
@@ -33,12 +41,20 @@
       </inertial>
     </link>
-    <joint name="joint_${name}_wheel" type="continuous">
-      <parent link="${parent}"/>
-      <child link="${name}_wheel"/>
-      <insert_block name="origin" />
-      <axis xyz="0 1 0" rpy="0 0 0" />
-      <limit effort="100" velocity="100"/>
-      <joint_properties damping="0.0" friction="0.0"/>
+     <joint name="joint_${name}_wheel_cover" type="fixed">
+      <parent link="${name}_wheel"/>
+      <child link="${name}_wheel_cover"/>
+      <origin xyz="0 0 0" rpy="0 0 0"/>
     </joint>
+     <link name="${name}_wheel_cover">
+      <visual>
+		<origin xyz="0 0 0" rpy="${reflect*PI} 0 0" />
+        <geometry>
+          <mesh filename="package://summit_xl_description/meshes/wheels/rubber_wheel_cover.stl" />
+        </geometry>
+        <material name="white">
+           <color rgba="0.6 0.6 0.6 1"/>
+        </material>
+      </visual>
+     </link>
     <!-- Transmission is important to link the joints and the controller (see summit_xl_control/config/summit_xl_control.yaml)-->
     <transmission name="${name}_wheel_joint_trans">
