Commit message: Visulization in Gazebo almost done. Chassis origin and STL's corrected.

File: summit_xl_description/robots/summit_xl_hq.urdf.xacro (robot description, xacro)
@@ -2,18 +2,15 @@
 <robot name="summit_xl" xmlns:xacro="http://www.ros.org/wiki/xacro">
   <!-- Import all Gazebo-customization elements, including Gazebo colors -->
-  <xacro:include filename="$(find summit_xl_description)/urdf/summit_xl_hq.gazebo" />
+  <xacro:include filename="$(find summit_xl_description)/urdf/bases/summit_xl_base.gazebo.xacro" />
   <xacro:include filename="$(find summit_xl_description)/urdf/bases/summit_xl_base.urdf.xacro" />
   <xacro:include filename="$(find summit_xl_description)/urdf/wheels/rubber_wheel.urdf.xacro" />
   <xacro:include filename="$(find summit_xl_description)/urdf/sensors/kinect.urdf.xacro" />
+  <xacro:include filename="$(find summit_xl_description)/urdf/sensors/hokuyo_urg04lx.urdf.xacro" />
+  <xacro:include filename="$(find summit_xl_description)/urdf/sensors/hokuyo_utm30lx.urdf.xacro" />
   <!-- Robot mechanical and motor parameters -->
   <xacro:property name="PI" value="3.1415926535897931"/>
-  <xacro:property name="wheel_offset_x" value="0.223" />    <!-- x,y,z in base_link CS -->
-  <xacro:property name="wheel_offset_y" value="0.234" />
+  <xacro:property name="wheel_offset_x" value="0.229" />    <!-- x,y,z in base_link CS -->
+  <xacro:property name="wheel_offset_y" value="0.234" />    <!-- y distance between base_link and the center of the wheel -->
   <xacro:property name="wheel_offset_z" value="0.0" />
-  <xacro:property name="wheel_joint_damping" value="0.0" />
-  <xacro:property name="wheel_joint_friction" value="0.0" />
-  <xacro:property name="wheel_joint_effort_limit" value="100.0" />
-  <xacro:property name="wheel_joint_velocity_limit" value="100.0" />
-  <xacro:property name="wheel_mechanical_reduction" value="1.0" />
   <xacro:property name="ptz_joint_effort_limit" value="100.0" />
   <xacro:property name="ptz_joint_velocity_limit" value="100.0"/>
@@ -21,20 +18,19 @@
   <xacro:property name="ptz_joint_damping" value="0.1" />
   <xacro:property name="ptz_mechanical_reduction" value="1.0" />
-  <xacro:property name="rubber_wheels" value="true" />
-  <xacro:property name="rubber_wheels" value="true" />
-  <summit_xl_base name="summit_xl" />
+  <xacro:summit_xl_base name="summit_xl" publish_bf="true" />
+  <xacro:summit_xl_skid_gazebo/>
     <!-- WHEELS -->
-  <rubber_wheel name="front_right" parent="base_link" reflect="0">
+  <xacro:rubber_wheel name="front_right" parent="base_link" reflect="0" hq="true">
     <origin xyz="${wheel_offset_x} -${wheel_offset_y} ${wheel_offset_z}" rpy="0 0 0"/>
-  </rubber_wheel>
-  <rubber_wheel name="front_left" parent="base_link" reflect="1">
+  </xacro:rubber_wheel>
+  <xacro:rubber_wheel name="front_left" parent="base_link" reflect="1" hq="true">
     <origin xyz="${wheel_offset_x} ${wheel_offset_y} ${wheel_offset_z}" rpy="0 0 0"/>
-  </rubber_wheel>
-  <rubber_wheel name="back_left" parent="base_link" reflect="1">
+  </xacro:rubber_wheel>
+  <xacro:rubber_wheel name="back_left" parent="base_link" reflect="1" hq="true">
     <origin xyz="-${wheel_offset_x} ${wheel_offset_y} ${wheel_offset_z}" rpy="0 0 0"/>
-  </rubber_wheel>
-  <rubber_wheel name="back_right" parent="base_link" reflect="0">
+  </xacro:rubber_wheel>
+  <xacro:rubber_wheel name="back_right" parent="base_link" reflect="0" hq="true">
     <origin xyz="-${wheel_offset_x} -${wheel_offset_y} ${wheel_offset_z}" rpy="0 0 0"/>
-  </rubber_wheel>
+  </xacro:rubber_wheel>
   <!-- IMU SENSOR -->
   <joint name="imu_joint" type="fixed">
@@ -63,9 +59,9 @@
       </collision>
   </link>
-  <sensor_kinect name="kinect1" parent="base_link">
+  <xacro:sensor_kinect name="kinect1" parent="base_link">
     <origin xyz="0.33 0 0.33" rpy="0 0 0"/>
-  </sensor_kinect>
-  <sensor_kinect name="kinect2" parent="base_link">
-    <origin xyz="0.33 0 0.43" rpy="0 0 0"/>
-  </sensor_kinect>
+  </xacro:sensor_kinect>
+  <xacro:sensor_hokuyo_utm30lx name="hokuyo" parent="base_link">
+    <origin xyz="0.0 0.0 0.36" rpy="0 0 0"/>
+  </xacro:sensor_hokuyo_utm30lx>
 </robot>

File: summit_xl_description/urdf/bases/summit_xl_base.gazebo.xacro (robot description, xacro)
@@ -1,16 +1,17 @@
 <?xml version="1.0"?>
-<robot>
-  <!-- ros_control plugin -->
-  <gazebo>
-    <plugin name="ros_control" filename="libgazebo_ros_control.so">
-       <robotNamespace>$(arg namespace)</robotNamespace>
-       <robotParam>$(arg namespace)/robot_description</robotParam>
-       <controlPeriod>0.003</controlPeriod>
-	     <robotSimType>gazebo_ros_control/DefaultRobotHWSim</robotSimType>
-    </plugin>
-  </gazebo>
-  <gazebo>
-    <plugin name="skid_steer_drive_controller" filename="libgazebo_ros_skid_steer_drive.so">
-			<robotNamespace>$(arg namespace)</robotNamespace>
+<robot xmlns:xacro="http://ros.org/wiki/xacro">
+  <!-- ros_control skid steer plugin -->
+  <xacro:macro name="summit_xl_skid_gazebo">
+    <gazebo>
+      <plugin name="ros_control" filename="libgazebo_ros_control.so">
+        <robotNamespace>$(arg namespace)</robotNamespace>
+        <robotParam>$(arg namespace)/robot_description</robotParam>
+        <controlPeriod>0.003</controlPeriod>
+	    <robotSimType>gazebo_ros_control/DefaultRobotHWSim</robotSimType>
+      </plugin>
+    </gazebo>
+    <gazebo>
+      <plugin name="skid_steer_drive_controller" filename="libgazebo_ros_skid_steer_drive.so">
+		<robotNamespace>$(arg namespace)</robotNamespace>
 	    <updateRate>100.0</updateRate>
 	    <leftFrontJoint>joint_front_left_wheel</leftFrontJoint>
@@ -27,35 +28,21 @@
 	    <odometryFrame>$(arg namespace)/odom</odometryFrame>
 	    <broadcastTF>1</broadcastTF>
-    </plugin>
-  </gazebo>
+      </plugin>
+    </gazebo>
+  </xacro:macro>
   <gazebo reference="base_footprint">
     <material>Gazebo/Green</material>
   </gazebo>
   <gazebo reference="base_link">
+    <material>Gazebo/Black</material>
+  </gazebo>
+  <gazebo reference="logos_link">
     <material>Gazebo/Red</material>
   </gazebo>
-  <gazebo reference="back_left_wheel">
-    <mu1 value="4.0"/> <!-- 2.0 -->
-    <mu2 value="1.0"/> <!-- 0.5 -->
-    <fdir1 value="1 0 0"/>
+  <gazebo reference="covers_link">
     <material>Gazebo/Grey</material>
   </gazebo>
-  <gazebo reference="back_right_wheel">
-    <mu1 value="4.0"/> <!-- 2.0 -->
-    <mu2 value="1.0"/> <!-- 0.5 -->
-    <fdir1 value="1 0 0"/>
-    <material>Gazebo/Grey</material>
-  </gazebo>
-  <gazebo reference="front_left_wheel">
-    <mu1 value="4.0"/> <!-- 2.0 -->
-    <mu2 value="1.0"/> <!-- 0.5 -->
-    <fdir1 value="1 0 0"/>
-    <material>Gazebo/Grey</material>
-  </gazebo>
-  <gazebo reference="front_right_wheel">
-    <mu1 value="4.0"/> <!-- 2.0 -->
-    <mu2 value="1.0"/> <!-- 0.5 -->
-    <fdir1 value="1 0 0"/>
-    <material>Gazebo/Grey</material>
+  <gazebo reference="back_left_wheel_cover">
+     <material>Gazebo/Red</material>
   </gazebo>
   <!-- camera -->
@@ -103,42 +90,4 @@
     </sensor>
   </gazebo>
-  <!-- hokuyo -->
-  <gazebo reference="hokuyo_laser_link">
-    <!-- sensor type="gpu_ray" name="head_hokuyo_sensor" -->
-    <sensor type="ray" name="head_hokuyo_sensor">
-      <pose>0 0 0 0 0 0</pose>
-      <visualize>false</visualize>
-      <update_rate>30</update_rate>
-      <ray>
-        <scan>
-          <horizontal>
-            <!-- samples>720</samples>
-            <resolution>1</resolution>
-            <min_angle>-1.570796</min_angle>
-            <max_angle>1.570796</max_angle -->
-           <samples>1081</samples>
-           <resolution>1</resolution>
-           <min_angle>2.35619449</min_angle>  <!-- +/-135 deg -->
-           <max_angle>-2.35619449</max_angle>
-          </horizontal>
-        </scan>
-        <range>
-          <min>0.10</min>
-          <max>30.0</max>
-          <resolution>0.01</resolution>
-        </range>
-        <noise>
-          <type>gaussian</type>
-          <mean>0.0</mean>
-          <stddev>0.01</stddev>
-        </noise>
-      </ray>
-      <!-- plugin name="gazebo_ros_head_hokuyo_controller" filename="libgazebo_ros_gpu_laser.so" -->
-      <plugin name="gazebo_ros_head_hokuyo_controller" filename="libgazebo_ros_laser.so">
-        <topicName>scan</topicName>
-        <frameName>hokuyo_laser_link</frameName>
-      </plugin>
-    </sensor>
-  </gazebo>
 <!--
   <gazebo>

File: summit_xl_description/urdf/bases/summit_xl_base.urdf.xacro (robot description, xacro)
@@ -1,27 +1,8 @@
 <?xml version="1.0"?>
 <robot name="summit_xl" xmlns:xacro="http://www.ros.org/wiki/xacro">
-  <!-- Import all Gazebo-customization elements, including Gazebo colors -->
-  <xacro:include filename="$(find summit_xl_description)/urdf/summit_xl.gazebo"/>
-  <xacro:macro name="summit_xl_base" params="name">
-  <!-- Robot mechanical and motor parameters -->
-  <xacro:property name="PI" value="3.1415926535897931"/>
-  <xacro:property name="wheel_offset_x" value="0.223" />    <!-- x,y,z in base_footprint CS -->
-  <xacro:property name="wheel_offset_y" value="0.154" />
-  <xacro:property name="wheel_offset_z" value="0.0" />
-  <xacro:property name="wheel_joint_damping" value="0.0" />
-  <xacro:property name="wheel_joint_friction" value="0.0" />
-  <xacro:property name="wheel_joint_effort_limit" value="200.0" />
-  <xacro:property name="wheel_joint_velocity_limit" value="200.0" />
-  <xacro:property name="wheel_mechanical_reduction" value="1.0" />
-  <xacro:property name="wheel_width" value="0.175" />
-  <xacro:property name="ptz_joint_effort_limit" value="100.0" />
-  <xacro:property name="ptz_joint_velocity_limit" value="100.0"/>
-  <xacro:property name="ptz_joint_friction" value="0.1" />
-  <xacro:property name="ptz_joint_damping" value="0.1" />
-  <xacro:property name="ptz_mechanical_reduction" value="1.0" />
+  <xacro:macro name="summit_xl_base" params="name publish_bf">
   <!-- BASE FOOTPRINT -->
-  <!-- base_footprint is a fictitious link(frame) that is on the ground right below base_link origin,
-             navigation stack depends on this frame -->
-  <link name="base_footprint">
+  <xacro:if value="true">
+    <link name="base_footprint">
       <visual>
           <origin xyz="0 0 0" rpy="0 0 0" />
@@ -30,19 +11,20 @@
           </geometry>
       </visual>
+<!--
       <collision>
           <origin xyz="0 0 0" rpy="0 0 0" />
           <geometry>
             <box size="0.001 0.001 0.001" />
-         </geometry>
-     </collision>
-  </link>
-  <joint name="base_footprint_joint" type="fixed">
-     <!-- NB While you would think this would make it go up, it is oddly reversed.
-      This moves the joint to 0,0,0 where we want it for rviz, etc. -->
-     <origin xyz="0 0 0.050" rpy="0 0 0" />
-     <parent link="base_footprint"/>
-     <child link="base_link" />
-  </joint>
-  <!-- BASE_LINK (RED) -->
+          </geometry>
+      </collision>
+-->
+    </link>
+    <joint name="base_footprint_joint" type="fixed">
+      <origin xyz="0 0 ${wheel_radius}" rpy="0 0 0" /> <!-- ${wheel_radius} property must be defined inside wheel description -->
+      <parent link="base_footprint"/>
+      <child link="base_link" />
+    </joint>
+  </xacro:if>
+  <!-- BASE_LINK -->
   <link name="base_link">
     <inertial>
@@ -54,15 +36,51 @@
        <origin xyz="0 0 0" rpy="0 0 0" />
        <geometry>
-	     <mesh filename="package://summit_xl_description/meshes/bases/summit_xl_chassis.dae"/>
+	     <mesh filename="package://summit_xl_description/meshes/bases/summit_xl_chassis.stl"/>
        </geometry>
+       <material name="darkgrey">
+         <color rgba="0.1 0.1 0.1 1"/>
+       </material>
     </visual>
     <collision>
        <origin xyz="0 0 0" rpy="0 0 0 " />
        <geometry>
-         <mesh filename="package://summit_xl_description/meshes/bases/summit_xl_chassis.dae"/>
-	     <!-- box size = "0.750 0.4 0.3"/ -->
+         <mesh filename="package://summit_xl_description/meshes/bases/summit_xl_chassis.stl"/>
        </geometry>
     </collision>
   </link>
+  <!-- COVERS AND SUSPENSIONS -->
+  <joint name="covers_joint" type="fixed">
+     <origin xyz="0 0 0" rpy="0 0 0" />
+     <parent link="base_link"/>
+     <child link="covers_link" />
+  </joint>
+  <link name="covers_link">
+    <visual>
+       <origin xyz="0 0 0" rpy="0 0 0" />
+       <geometry>
+	     <mesh filename="package://summit_xl_description/meshes/bases/summit_xl_covers.stl"/>
+       </geometry>
+       <material name="silver">
+         <color rgba="0.6 0.6 0.6 1"/>
+       </material>
+    </visual>
+  </link>
+  <!-- LOGOS -->
+  <joint name="logos_joint" type="fixed">
+     <origin xyz="0 0 0" rpy="0 0 0" />
+     <parent link="base_link"/>
+     <child link="logos_link" />
+  </joint>
+  <link name="logos_link">
+    <visual>
+       <origin xyz="0 0 0" rpy="0 0 0" />
+       <geometry>
+	     <mesh filename="package://summit_xl_description/meshes/bases/summit_xl_logos.stl" scale="1.001 1.001 1.001"/> <!-- Scaled a little bit up to avoid visualization problems -->
+       </geometry>
+       <material name="red">
+         <color rgba="0.8 0.1 0.1 1"/>
+       </material>
+    </visual>
+  </link>
   </xacro:macro>
 </robot>

File: summit_xl_description/urdf/sensors/hokuyo_utm30lx.urdf.xacro (robot description, xacro)
@@ -1,6 +1,5 @@
 <?xml version="1.0"?>
-<robot name="sensor_hokuyo" xmlns:xacro="http://ros.org/wiki/xacro">
-	<xacro:property name="M_PI" value="3.1415926535897931" />
-  <xacro:macro name="hokuyo_sensor" params="name parent *origin">
+<robot name="sensor_hokuyo_utm30lx" xmlns:xacro="http://ros.org/wiki/xacro">
+  <xacro:macro name="sensor_hokuyo_utm30lx" params="name parent *origin">
     <joint name="${name}_laser_joint" type="fixed">
       <!-- FRONT MOUNT -->
@@ -11,26 +10,26 @@
       <parent link="${parent}"/>
       <child link="${name}_laser_link"/>
-		</joint>
-		<link name="${name}_laser_link">
-			<collision>
-				<origin xyz="0 0 0" rpy="0 0 0"/>
-				<geometry>
-					<box size="0.1 0.1 0.1"/>
-				</geometry>
-			</collision>
-			<visual>
-				<origin xyz="0 0 0" rpy="0 0 0"/>
-				<geometry>
-					<mesh filename="package://summit_xl_description/meshes/hokuyo-utm30-lx.dae"/>
-				</geometry>
-			</visual>
-			<inertial>
-				<mass value="1e-5" />
-				<origin xyz="0 0 0" rpy="0 0 0"/>
-				<inertia ixx="1e-6" ixy="0" ixz="0" iyy="1e-6" iyz="0" izz="1e-6" />
-			</inertial>
-		</link>
-		<!-- Kinect sensor for simulation -->
-		<kinect_sim_3dsensor/>
+	</joint>
+	<link name="${name}_laser_link">
+		<collision>
+			<origin xyz="0 0 0" rpy="0 0 0"/>
+			<geometry>
+				<box size="0.1 0.1 0.08"/>
+			</geometry>
+		</collision>
+		<visual>
+			<origin xyz="0 0 0" rpy="0 0 0"/>
+			<geometry>
+	     		<mesh filename="package://summit_xl_description/meshes/sensors/hokuyo_utm_30lx.dae"/>
+			</geometry>
+		</visual>
+		<inertial>
+			<mass value="1e-5" />
+			<origin xyz="0 0 0" rpy="0 0 0"/>
+			<inertia ixx="1e-6" ixy="0" ixz="0" iyy="1e-6" iyz="0" izz="1e-6" />
+		</inertial>
+	</link>
+	<!-- Hokuyo sensor for simulation -->
+	<hokuyo_sim_sensor/>
   </xacro:macro>
   <xacro:macro name="hokuyo_sim_sensor">
@@ -61,9 +60,9 @@
 				</ray>
 				<plugin name="gazebo_ros_head_hokuyo_controller" filename="libgazebo_ros_laser.so">
-					<topicName>scan</topicName>
+					<topicName>${name}/scan</topicName>
 					<frameName>${name}_laser_link</frameName>
 				</plugin>
 			</sensor>
-		</gazebo>
+	</gazebo>
   </xacro:macro>
 </robot>

File: summit_xl_description/urdf/sensors/kinect.urdf.xacro (robot description, xacro)
@@ -1,6 +1,5 @@
 <?xml version="1.0"?>
 <robot name="sensor_kinect" xmlns:xacro="http://ros.org/wiki/xacro">
-	<xacro:property name="M_PI" value="3.1415926535897931" />
-  <!-- Parameterised in part by the values in turtlebot_properties.urdf.xacro -->
+  <xacro:property name="M_PI" value="3.1415926535897931" />
   <xacro:macro name="sensor_kinect" params="name parent *origin">
     <joint name="${name}_camera_rgb_joint" type="fixed">
@@ -93,5 +92,5 @@
   </xacro:macro>
   	<xacro:macro name="kinect_sim_3dsensor">
-    <gazebo reference="camera_link">
+    <gazebo reference="${name}_camera_link">
       <sensor type="depth" name="camera">
         <always_on>true</always_on>

File: summit_xl_description/urdf/wheels/omni_wheel.urdf.xacro (robot description, xacro)
@@ -1,11 +1,9 @@
 <?xml version="1.0"?>
 <robot name="wheel" xmlns:xacro="http://www.ros.org/wiki/xacro">
+  <xacro:property name="M_PI" value="3.1415926535897931" />
   <!-- Wheels -->
-  <property name="wheel_radius" value="0.125" />
-  <property name="wheel_height" value="0.14" />
-  <property name="wheel_mass" value="2.5" /> <!-- in kg-->
-  <property name="base_x_origin_to_wheel_origin" value="0.22911" />
-  <property name="base_y_origin_to_wheel_origin" value="0.23350" />
-  <property name="base_z_origin_to_wheel_origin" value="0.0" />
+  <property name="wheel_radius" value="0.117" />
+  <property name="wheel_height" value="0.12" />
+  <property name="wheel_mass" value="6.5" /> <!-- in kg-->
   <macro name="cylinder_inertia" params="m r h">
     <inertia  ixx="${m*(3*r*r+h*h)/12}" ixy = "0" ixz = "0"
@@ -13,17 +11,35 @@
               izz="${m*r*r/2}" />
   </macro>
-  <xacro:macro name="wheel" params="fb lr parent translateX translateY flipY"> <!--fb : front, back ; lr: left, right -->
-    <link name="${fb}_${lr}_wheel">
+  <xacro:macro name="rubber_wheel" params="name parent *origin reflect hq">
+    <joint name="joint_${name}_wheel" type="continuous">
+      <parent link="${parent}"/>
+      <child link="${name}_wheel"/>
+      <insert_block name="origin" />
+      <axis xyz="0 1 0" rpy="0 0 0" />
+      <limit effort="100" velocity="100"/>
+      <joint_properties damping="0.0" friction="0.0"/>
+    </joint>
+    <link name="${name}_wheel">
       <visual>
-        <origin xyz="0 0 0" rpy="${flipY*M_PI*2} 0 0" />
-        <geometry>
-          <mesh filename="package://summit_xl_description/meshes/summit_xl_wheel_hq.stl" />
-        </geometry>
-        <material name="DarkGray" />
+        <xacro:if value="${hq}">
+          <origin xyz="0 0 0" rpy="0 0 0" />
+          <geometry>
+            <mesh filename="package://summit_xl_description/meshes/wheels/omni_wheel.stl" />
+          </geometry>
+        </xacro:if>
+        <xacro:unless value="${hq}">
+          <origin xyz="0 0 0" rpy="0 0 0" />
+          <geometry>
+            <sphere radius="${wheel_radius}" />
+          </geometry>
+        </xacro:unless>
+        <material name="darkgrey">
+           <color rgba="0.2 0.2 0.2 1"/>
+        </material>
       </visual>
       <collision>
-        <origin xyz="0 0 0" rpy="${flipY*M_PI/2} 0 0" />
+		<origin xyz="0 0 0" rpy="0 0 0" />
         <geometry>
-          <cylinder length="${wheel_height}" radius="${wheel_radius}" />
+          <sphere radius="${wheel_radius}" />
         </geometry>
       </collision>
@@ -34,5 +50,30 @@
       </inertial>
     </link>
-    <gazebo reference="${fb}_${lr}_wheel">
+     <joint name="joint_${name}_wheel_cover" type="fixed">
+      <parent link="${name}_wheel"/>
+      <child link="${name}_wheel_cover"/>
+      <origin xyz="0 0 0" rpy="0 0 0"/>
+    </joint>
+     <link name="${name}_wheel_cover">
+      <visual>
+		<origin xyz="0 0 0" rpy="${reflect*PI} 0 0" />
+        <geometry>
+          <mesh filename="package://summit_xl_description/meshes/wheels/rubber_wheel_cover.stl" />
+        </geometry>
+        <material name="white">
+           <color rgba="0.6 0.6 0.6 1"/>
+        </material>
+      </visual>
+     </link>
+    <!-- Transmission is important to link the joints and the controller (see summit_xl_control/config/summit_xl_control.yaml)-->
+    <transmission name="${name}_wheel_joint_trans">
+      <type>transmission_interface/SimpleTransmission</type>
+      <joint name="joint_${name}_wheel" />
+      <actuator name="${name}_wheel_joint_motor">
+        <hardwareInterface>EffortJointInterface</hardwareInterface>
+        <mechanicalReduction>1</mechanicalReduction>
+      </actuator>
+    </transmission>
+    <gazebo reference="${name}_wheel">
 		<mu1 value="5.0"/>
 		<mu2 value="0.5"/>
@@ -40,24 +81,7 @@
 		<kd value="1.0" />
 		<fdir1 value="1 0 0"/>
-      <material>Gazebo/Grey</material>
+      <material>Gazebo/Gray</material>
       <turnGravityOff>false</turnGravityOff>
     </gazebo>
-    <joint name="joint_${fb}_${lr}_wheel" type="continuous">
-      <parent link="${parent}"/>
-      <child link="${fb}_${lr}_wheel"/>
-      <origin xyz="${translateX * base_x_origin_to_wheel_origin} ${translateY * base_y_origin_to_wheel_origin} ${base_z_origin_to_wheel_origin}" rpy="0 0 0" />
-      <axis xyz="0 1 0" rpy="0 0 0" />
-      <limit effort="100" velocity="100"/>
-      <joint_properties damping="0.0" friction="0.0"/>
-    </joint>
-    <!-- Transmission is important to link the joints and the controller (see summit_xl_control/config/summit_xl_control.yaml)-->
-    <transmission name="${fb}_${lr}_wheel_joint_trans">
-      <type>transmission_interface/SimpleTransmission</type>
-      <joint name="joint_${fb}_${lr}_wheel" />
-      <actuator name="${fb}_${lr}_wheel_joint_motor">
-        <hardwareInterface>EffortJointInterface</hardwareInterface>
-        <mechanicalReduction>1</mechanicalReduction>
-      </actuator>
-    </transmission>
   </xacro:macro>
 </robot>
