Commit message: Visulization in Gazebo almost done. Chassis origin and STL's corrected.

File: summit_xl_description/urdf/wheels/rubber_wheel.urdf.xacro (robot description, xacro)
@@ -1,14 +1,16 @@
 <?xml version="1.0"?>
 <robot name="wheel" xmlns:xacro="http://www.ros.org/wiki/xacro">
+  <xacro:property name="M_PI" value="3.1415926535897931" />
   <!-- Wheels -->
-  <property name="wheel_radius" value="0.125" />
-  <property name="wheel_height" value="0.14" />
-  <property name="wheel_mass" value="2.5" /> <!-- in kg-->
-  <macro name="cylinder_inertia" params="m r h">
+  <property name="wheel_radius" value="0.117" />
+  <property name="wheel_height" value="0.12" />
+  <property name="wheel_mass" value="6.5" /> <!-- in kg-->
+  <xacro:macro name="cylinder_inertia" params="m r h">
     <inertia  ixx="${m*(3*r*r+h*h)/12}" ixy = "0" ixz = "0"
               iyy="${m*(3*r*r+h*h)/12}" iyz = "0"
               izz="${m*r*r/2}" />
-  </macro>
-  <xacro:macro name="rubber_wheel" params="name parent *origin reflect">
+  </xacro:macro>
+  <xacro:macro name="rubber_wheel" params="name parent *origin reflect hq">
+<!--WHEEL TIRE -->
     <joint name="joint_${name}_wheel" type="continuous">
       <parent link="${parent}"/>
@@ -21,8 +23,18 @@
     <link name="${name}_wheel">
       <visual>
-		<origin xyz="0 0 0" rpy="0 0 0" />
-        <geometry>
-          <mesh filename="package://summit_xl_description/meshes/wheels/rubber_wheel.stl" />
-        </geometry>
+        <!-- HIGH RESOLUTION WHEELS -->
+        <xacro:if value="${hq}">
+          <origin xyz="0 0 0" rpy="0 0 0" />
+          <geometry>
+            <mesh filename="package://summit_xl_description/meshes/wheels/rubber_wheel.stl" />
+          </geometry>
+        </xacro:if>
+       <!-- LOW RESOLUTION WHEELS -->
+        <xacro:unless value="${hq}">
+          <origin xyz="0 0 0" rpy="${M_PI/2} 0 0" />
+          <geometry>
+            <cylinder length="${wheel_height}" radius="${wheel_radius}" />
+          </geometry>
+        </xacro:unless>
         <material name="darkgrey">
            <color rgba="0.2 0.2 0.2 1"/>
@@ -30,5 +42,5 @@
       </visual>
       <collision>
-		<origin xyz="0 0 0" rpy="0 0 0" />
+		<origin xyz="0 0 0" rpy="${M_PI/2} 0 0" />
         <geometry>
           <cylinder length="${wheel_height}" radius="${wheel_radius}" />
@@ -41,5 +53,6 @@
       </inertial>
     </link>
-     <joint name="joint_${name}_wheel_cover" type="fixed">
+<!-- WHEEL COVERS -->
+    <joint name="joint_${name}_wheel_cover" type="fixed">
       <parent link="${name}_wheel"/>
       <child link="${name}_wheel_cover"/>
@@ -52,8 +65,17 @@
           <mesh filename="package://summit_xl_description/meshes/wheels/rubber_wheel_cover.stl" />
         </geometry>
-        <material name="white">
+        <material name="lightgrey">
            <color rgba="0.6 0.6 0.6 1"/>
         </material>
       </visual>
+<!-- MOTOR VISUAL -->
+<!--
+      <visual>
+        <origin xyz="0 0 0" rpy="${M_PI/2} 0 0" />
+        <geometry>
+          <cylinder length="${wheel_height}" radius="0.05" />
+        </geometry>
+      </visual>
+-->
      </link>
     <!-- Transmission is important to link the joints and the controller (see summit_xl_control/config/summit_xl_control.yaml)-->
@@ -72,7 +94,11 @@
 		<kd value="1.0" />
 		<fdir1 value="1 0 0"/>
-      <material>Gazebo/Gray</material>
       <turnGravityOff>false</turnGravityOff>
     </gazebo>
+<!--
+    <gazebo reference="${name}_wheel_cover">
+      <material>Gazebo/Red</material>
+    </gazebo>
+-->
   </xacro:macro>
 </robot>

Commit message: Not anymore multi.

File: summit_xl_description/robots/summit_xl_hq.urdf.xacro (robot description, xacro)
@@ -19,5 +19,5 @@
   <xacro:property name="ptz_mechanical_reduction" value="1.0" />
 -->
-  <xacro:summit_xl_base name="summit_xl" publish_bf="true" />
+  <xacro:summit_xl_base name="summit_xl" publish_bf="false" hq="true" />
   <xacro:summit_xl_skid_gazebo/>
     <!-- WHEELS -->
@@ -60,7 +60,9 @@
       </collision>
   </link>
+<!--
   <xacro:sensor_hokuyo_urg04lx name="hokuyo1" parent="base_link">
     <origin xyz="0.0 0.0 0.36" rpy="0 0 0"/>
   </xacro:sensor_hokuyo_urg04lx>
+-->
   <xacro:sensor_hokuyo_utm30lx name="hokuyo2" parent="base_link">
     <origin xyz="0.0 0.0 0.46" rpy="0 0 0"/>

File: summit_xl_description/urdf/bases/summit_xl_base.gazebo.xacro (robot description, xacro)
@@ -5,6 +5,6 @@
     <gazebo>
       <plugin name="ros_control" filename="libgazebo_ros_control.so">
-        <robotNamespace>$(arg namespace)</robotNamespace>
-        <robotParam>$(arg namespace)/robot_description</robotParam>
+        <robotNamespace>/summit_xl</robotNamespace>
+        <robotParam>robot_description</robotParam>
         <controlPeriod>0.003</controlPeriod>
 	    <robotSimType>gazebo_ros_control/DefaultRobotHWSim</robotSimType>
@@ -13,5 +13,5 @@
     <gazebo>
       <plugin name="skid_steer_drive_controller" filename="libgazebo_ros_skid_steer_drive.so">
-		<robotNamespace>$(arg namespace)</robotNamespace>
+		<robotNamespace>/summit_xl</robotNamespace>
 	    <updateRate>100.0</updateRate>
 	    <leftFrontJoint>joint_front_left_wheel</leftFrontJoint>
@@ -19,13 +19,13 @@
 	    <leftRearJoint>joint_back_left_wheel</leftRearJoint>
 	    <rightRearJoint>joint_back_right_wheel</rightRearJoint>
-	    <wheelSeparation>0.308</wheelSeparation>
+	    <wheelSeparation>0.472</wheelSeparation>
 	    <wheelDiameter>0.125</wheelDiameter>
-	    <robotBaseFrame>$(arg namespace)/base_footprint</robotBaseFrame>
+	    <robotBaseFrame>base_footprint</robotBaseFrame>
 	    <torque>25</torque>
 	    <topicName>cmd_vel</topicName>
 	    <commandTopic>summit_xl_robot_control/command</commandTopic>
 	    <odometryTopic>odom</odometryTopic>
-	    <odometryFrame>$(arg namespace)/odom</odometryFrame>
-	    <broadcastTF>1</broadcastTF>
+	    <odometryFrame>/odom</odometryFrame>
+	    <broadcastTF>true</broadcastTF>
       </plugin>
     </gazebo>
@@ -86,5 +86,4 @@
   </gazebo>
 -->
-<!--
   <gazebo>
     <plugin name="ros_imu" filename="libgazebo_ros_imu.so">
@@ -95,4 +94,3 @@
     </plugin>
   </gazebo>
--->
 </robot>

File: summit_xl_description/urdf/bases/summit_xl_base.urdf.xacro (robot description, xacro)
@@ -1,5 +1,5 @@
 <?xml version="1.0"?>
 <robot name="summit_xl" xmlns:xacro="http://www.ros.org/wiki/xacro">
-  <xacro:macro name="summit_xl_base" params="name publish_bf">
+  <xacro:macro name="summit_xl_base" params="name publish_bf hq">
   <!-- Robot mechanical and motor parameters -->
   <xacro:property name="PI" value="3.1415926535897931"/>
@@ -41,7 +41,14 @@
     <visual>
        <origin xyz="0 0 0" rpy="0 0 0" />
+       <xacro:if value="${hq}">
+       <geometry>
+	     <mesh filename="package://summit_xl_description/meshes/bases/summit_xl_chassis.stl"/>
+       </geometry>
+       </xacro:if>
+       <xacro:unless value="${hq}">
        <geometry>
 	     <mesh filename="package://summit_xl_description/meshes/bases/summit_xl_chassis_simple.stl"/>
        </geometry>
+       </xacro:unless>
        <material name="darkgrey">
          <color rgba="0.1 0.1 0.1 1"/>
@@ -56,5 +63,5 @@
   </link>
   <!-- COVERS AND SUSPENSIONS -->
-<!--
+  <xacro:if value="${hq}">
   <joint name="covers_joint" type="fixed">
      <origin xyz="0 0 0" rpy="0 0 0" />
@@ -73,5 +80,5 @@
     </visual>
   </link>
--->
+  </xacro:if>
   <!-- LOGOS -->
   <joint name="logos_joint" type="fixed">

Commit message: summit_xl_description: fixing axis model

File: summit_xl_description/robots/summit_xl_hq.urdf.xacro (robot description, xacro)
@@ -7,4 +7,5 @@
   <xacro:include filename="$(find summit_xl_description)/urdf/sensors/hokuyo_urg04lx.urdf.xacro" />
   <xacro:include filename="$(find summit_xl_description)/urdf/sensors/hokuyo_utm30lx.urdf.xacro" />
+  <xacro:include filename="$(find summit_xl_description)/urdf/sensors/axis.urdf.xacro" />
   <!-- Robot mechanical and motor parameters -->
   <xacro:property name="PI" value="3.1415926535897931"/>
@@ -68,3 +69,6 @@
     <origin xyz="0.0 0.0 0.46" rpy="0 0 0"/>
   </xacro:sensor_hokuyo_utm30lx>
+  <xacro:sensor_axis name="camera" parent="base_link">
+		<origin xyz="0.19 0 0.17" rpy="0 ${15*PI/180} 0"/>
+  </xacro:sensor_axis>
 </robot>

File: summit_xl_description/urdf/sensors/axis.urdf.xacro (robot description, xacro)
@@ -14,7 +14,7 @@
 				<insert_block name="origin"/>
 	      <parent link="${parent}"/>
-	      <child link="${name}_base_link"/>
+	      <child link="${name}_link"/>
 	  </joint>
-    <link name="${name}_base_link">
+    <link name="${name}_link">
       <inertial>
 				<origin xyz="0.03 0.0 -0.3" rpy="0 0 0"/>
@@ -25,6 +25,9 @@
       <visual>
 	      <origin xyz="0.03 0.0 -0.3" rpy="0 0 0"/> <!-- to center the axis model -->
+	      <material name="axis_color">
+           <color rgba="0.1 0.1 0.1 1"/>
+        </material>
 	      <geometry>
-					<mesh filename= "package://summit_xl_description/meshes/xl_fotonic/axis_p5512.dae" scale="1.0 1.0 1.0"/>
+					<mesh filename= "package://summit_xl_description/meshes/xl_fotonic/axis_p5512.stl" scale="1.0 1.0 1.0"/>
 	      </geometry>
 	    </visual>
@@ -32,12 +35,12 @@
 	      <origin xyz="0.03 0.0 -0.3" rpy="0 0 0"/>
 	      <geometry>
-	        <mesh filename= "package://summit_xl_description/meshes/xl_fotonic/axis_p5512.dae" scale="1.0 1.0 1.0"/>
+	        <mesh filename= "package://summit_xl_description/meshes/xl_fotonic/axis_p5512.stl" scale="1.0 1.0 1.0"/>
 	      </geometry>
 	    </collision>
     </link>
-	  <joint name="${name}_pan_joint" type="continuous">
+	  <joint name="joint_${name}_pan" type="continuous">
 	     <axis xyz="0 0 1" />
-	     <origin xyz="0.0 0.0 0.15"/>
-	     <parent link="${name}_base_link"/>
+	     <origin xyz="0.0 0.0 0.1"/>
+	     <parent link="${name}_link"/>
 	     <child link="${name}_pan_link"/>
 	     <limit effort="${ptz_joint_effort_limit}" velocity="${ptz_joint_velocity_limit}" lower="-3.1416" upper="3.1416"/>
@@ -53,5 +56,5 @@
 	  <transmission name="${name}_pan_trans">
 		 <type>transmission_interface/SimpleTransmission</type>
-	     <joint name="${name}_pan_joint" />
+	     <joint name="joint_${name}_pan" />
 	     <actuator name="pan_motor">
 			   <hardwareInterface>EffortJointInterface</hardwareInterface>
@@ -59,5 +62,5 @@
 	     </actuator>
 	  </transmission>
-	  <joint name="${name}_tilt_joint" type="continuous">
+	  <joint name="joint_${name}_tilt" type="continuous">
 	     <axis xyz="0 1 0" />
 	     <origin xyz="0.0 0.0 0.0"/>
@@ -76,5 +79,5 @@
 	  <transmission name="${name}_tilt_trans">
 		 <type>transmission_interface/SimpleTransmission</type>
-	     <joint name="${name}_tilt_joint" />
+	     <joint name="joint_${name}_tilt" />
 	     <actuator name="tilt_motor">
 				 <hardwareInterface>EffortJointInterface</hardwareInterface>
@@ -82,4 +85,7 @@
 	     </actuator>
 	  </transmission>
+	  <gazebo reference="${name}_link">
+      <material>Gazebo/FlatBlack</material>
+    </gazebo>
 		<!-- Axis sensor for simulation -->
 		<sensor_axis_gazebo/>
@@ -97,5 +103,5 @@
 	        </image>
 	        <clip>
-	          <near>0.02</near>
+	          <near>0.03</near>
 	          <far>300</far>
 	        </clip>

Commit message: summit_xl_description: adding imu sensor

File: summit_xl_description/robots/summit_xl_hq.urdf.xacro (robot description, xacro)
@@ -8,4 +8,5 @@
   <xacro:include filename="$(find summit_xl_description)/urdf/sensors/hokuyo_utm30lx.urdf.xacro" />
   <xacro:include filename="$(find summit_xl_description)/urdf/sensors/axis.urdf.xacro" />
+  <xacro:include filename="$(find summit_xl_description)/urdf/sensors/imu.urdf.xacro" />
   <!-- Robot mechanical and motor parameters -->
   <xacro:property name="PI" value="3.1415926535897931"/>
@@ -20,7 +21,7 @@
   <xacro:property name="ptz_mechanical_reduction" value="1.0" />
 -->
-  <xacro:summit_xl_base name="summit_xl" publish_bf="false" hq="true" />
+  <xacro:summit_xl_base name="summit_xl" publish_bf="true" hq="true" />
   <xacro:summit_xl_skid_gazebo/>
-    <!-- WHEELS -->
+  <!-- WHEELS -->
   <xacro:rubber_wheel name="front_right" parent="base_link" reflect="0" hq="true">
     <origin xyz="${wheel_offset_x} -${wheel_offset_y} ${wheel_offset_z}" rpy="0 0 0"/>
@@ -35,30 +36,5 @@
     <origin xyz="-${wheel_offset_x} -${wheel_offset_y} ${wheel_offset_z}" rpy="0 0 0"/>
   </xacro:rubber_wheel>
-  <!-- IMU SENSOR -->
-  <joint name="imu_joint" type="fixed">
-      <axis xyz="1 0 0"/> <!-- 0 1 0 -->
-      <origin xyz="0 0 0.2825"/>
-      <parent link="base_link"/>
-      <child link="imu_link"/>
-  </joint>
-  <link name="imu_link">
-      <inertial>
-        <mass value="0.001"/>
-        <origin rpy="0 0 0" xyz="0 0 0"/>
-        <inertia ixx="0.0001" ixy="0" ixz="0" iyy="0.000001" iyz="0" izz="0.0001"/>
-      </inertial>
-      <visual>
-        <origin rpy="0 0 0" xyz="0 0 0"/>
-        <geometry>
-          <box size="0.001 0.001 0.001"/>
-        </geometry>
-      </visual>
-      <collision>
-        <origin rpy="0 0 0" xyz="0 0 0"/>
-        <geometry>
-          <box size=".001 .001 .001"/>
-        </geometry>
-      </collision>
-  </link>
+	<!-- SENSORS -->
 <!--
   <xacro:sensor_hokuyo_urg04lx name="hokuyo1" parent="base_link">
@@ -72,3 +48,6 @@
 		<origin xyz="0.19 0 0.17" rpy="0 ${15*PI/180} 0"/>
   </xacro:sensor_axis>
+  <xacro:sensor_imu name="imu" parent="base_link">
+		<origin xyz="-0.18 0.0 0.170" rpy="0 0 0"/>
+  </xacro:sensor_imu>
 </robot>

File: summit_xl_description/urdf/bases/summit_xl_base.gazebo.xacro (robot description, xacro)
@@ -43,54 +43,3 @@
     <material>Gazebo/Grey</material>
   </gazebo>
-  <!-- camera -->
-  <!-- gazebo reference="camera_link" -->
-<!--
-  <gazebo reference="camera_tilt_link">
-    <mu1>0.2</mu1>
-    <mu2>0.2</mu2>
-    <material>Gazebo/Red</material>
-    <sensor type="camera" name="camera1">
-      <update_rate>30.0</update_rate>
-      <camera name="head">
-        <horizontal_fov>1.3962634</horizontal_fov>
-        <image>
-          <width>800</width>
-          <height>800</height>
-          <format>R8G8B8</format>
-        </image>
-        <clip>
-          <near>0.02</near>
-          <far>300</far>
-        </clip>
-        <noise>
-          <type>gaussian</type>
-          <mean>0.0</mean>
-          <stddev>0.007</stddev>
-        </noise>
-      </camera>
-      <plugin name="camera_controller" filename="libgazebo_ros_camera.so">
-        <alwaysOn>true</alwaysOn>
-        <updateRate>0.0</updateRate>
-        <cameraName>camera1</cameraName>
-        <imageTopicName>image_raw</imageTopicName>
-        <cameraInfoTopicName>camera_info</cameraInfoTopicName>
-        <frameName>camera_tilt_link</frameName>
-        <hackBaseline>0.07</hackBaseline>
-        <distortionK1>0.0</distortionK1>
-        <distortionK2>0.0</distortionK2>
-        <distortionK3>0.0</distortionK3>
-        <distortionT1>0.0</distortionT1>
-        <distortionT2>0.0</distortionT2>
-      </plugin>
-    </sensor>
-  </gazebo>
--->
-  <gazebo>
-    <plugin name="ros_imu" filename="libgazebo_ros_imu.so">
-       <topicName>imu_data</topicName>
-			 <bodyName>imu_link</bodyName>
-			 <serviceName>imu_service</serviceName>
-       <gaussianNoise>0.005</gaussianNoise>
-    </plugin>
-  </gazebo>
 </robot>

Commit message: summit_xl_description: fixing hokuyo position on the robot model

File: summit_xl_description/robots/summit_xl_hq.urdf.xacro (robot description, xacro)
@@ -14,11 +14,4 @@
   <xacro:property name="wheel_offset_y" value="0.234" />    <!-- y distance between base_link and the center of the wheel -->
   <xacro:property name="wheel_offset_z" value="0.0" />
-<!--
-  <xacro:property name="ptz_joint_effort_limit" value="100.0" />
-  <xacro:property name="ptz_joint_velocity_limit" value="100.0"/>
-  <xacro:property name="ptz_joint_friction" value="0.1" />
-  <xacro:property name="ptz_joint_damping" value="0.1" />
-  <xacro:property name="ptz_mechanical_reduction" value="1.0" />
--->
   <xacro:summit_xl_base name="summit_xl" publish_bf="true" hq="true" />
   <xacro:summit_xl_skid_gazebo/>
@@ -37,4 +30,7 @@
   </xacro:rubber_wheel>
 	<!-- SENSORS -->
+  <xacro:sensor_hokuyo_utm30lx name="hokuyo" parent="base_link">
+    <origin xyz="0.0 0.0 0.33" rpy="0 0 0"/>
+  </xacro:sensor_hokuyo_utm30lx>
 <!--
   <xacro:sensor_hokuyo_urg04lx name="hokuyo1" parent="base_link">
@@ -42,7 +38,4 @@
   </xacro:sensor_hokuyo_urg04lx>
 -->
-  <xacro:sensor_hokuyo_utm30lx name="hokuyo2" parent="base_link">
-    <origin xyz="0.0 0.0 0.46" rpy="0 0 0"/>
-  </xacro:sensor_hokuyo_utm30lx>
   <xacro:sensor_axis name="camera" parent="base_link">
 		<origin xyz="0.19 0 0.17" rpy="0 ${15*PI/180} 0"/>

Commit message: summit_xl_description: adding high_quality xacro parameter

File: summit_xl_description/robots/summit_xl_hq.urdf.xacro (robot description, xacro)
@@ -14,17 +14,19 @@
   <xacro:property name="wheel_offset_y" value="0.234" />    <!-- y distance between base_link and the center of the wheel -->
   <xacro:property name="wheel_offset_z" value="0.0" />
-  <xacro:summit_xl_base name="summit_xl" publish_bf="true" hq="true" />
+	<!-- Flag to select the high or low quality model -->
+  <xacro:property name="hq" value="true" />
+  <xacro:summit_xl_base name="summit_xl" publish_bf="true" hq="${hq}" />
   <xacro:summit_xl_skid_gazebo/>
   <!-- WHEELS -->
-  <xacro:rubber_wheel name="front_right" parent="base_link" reflect="0" hq="true">
+  <xacro:rubber_wheel name="front_right" parent="base_link" reflect="0" hq="${hq}">
     <origin xyz="${wheel_offset_x} -${wheel_offset_y} ${wheel_offset_z}" rpy="0 0 0"/>
   </xacro:rubber_wheel>
-  <xacro:rubber_wheel name="front_left" parent="base_link" reflect="1" hq="true">
+  <xacro:rubber_wheel name="front_left" parent="base_link" reflect="1" hq="${hq}">
     <origin xyz="${wheel_offset_x} ${wheel_offset_y} ${wheel_offset_z}" rpy="0 0 0"/>
   </xacro:rubber_wheel>
-  <xacro:rubber_wheel name="back_left" parent="base_link" reflect="1" hq="true">
+  <xacro:rubber_wheel name="back_left" parent="base_link" reflect="1" hq="${hq}">
     <origin xyz="-${wheel_offset_x} ${wheel_offset_y} ${wheel_offset_z}" rpy="0 0 0"/>
   </xacro:rubber_wheel>
-  <xacro:rubber_wheel name="back_right" parent="base_link" reflect="0" hq="true">
+  <xacro:rubber_wheel name="back_right" parent="base_link" reflect="0" hq="${hq}">
     <origin xyz="-${wheel_offset_x} -${wheel_offset_y} ${wheel_offset_z}" rpy="0 0 0"/>
   </xacro:rubber_wheel>
