Commit message: fixing summit XL omni movement. adding omni plugin for gazebo

File: summit_xl_description/robots/summit_xl_omni.urdf.xacro (robot description, xacro)
@@ -8,5 +8,5 @@
 	<xacro:include filename="$(find summit_xl_description)/urdf/bases/summit_xl_base.urdf.xacro" />
 	<!-- Import summit XL wheels -->
-	<xacro:include filename="$(find summit_xl_description)/urdf/wheels/rubber_wheel.urdf.xacro" />
+	<xacro:include filename="$(find summit_xl_description)/urdf/wheels/omni_wheel.urdf.xacro" />
 	<!-- Import all available sensors -->
 	<xacro:include filename="$(find summit_xl_description)/urdf/sensors/all_sensors.urdf.xacro" />
@@ -26,22 +26,22 @@
 	<!-- Here we create the robot elements using the xacro:macros imported at the beggining of this file -->
 	<!-- Summit XL base -->
-	<xacro:summit_xl_base name="summit_xl" publish_bf="true" hq="${hq}" />
-	<!-- Gazebo ros control pluggins -->
-	<xacro:ros_control/>
-	<!-- Gazebo skid steering pluggins -->
-	<xacro:skid_steering/>
+  <xacro:summit_xl_base name="summit_xl" publish_bf="true" hq="${hq}"/>
+  <!-- Gazebo ros control pluggins -->
+  <xacro:ros_control/>
+  <!-- Gazebo omni steering plugin -->
+	<xacro:omni_steering/>
 	<!-- WHEELS -->
-	<xacro:rubber_wheel name="front_right" parent="base_link" reflect="0" hq="${hq}">
+	<xacro:omni_wheel name="front_right" parent="base_link" reflect="false" hq="true">
 		<origin xyz="${wheel_offset_x} -${wheel_offset_y} ${wheel_offset_z}" rpy="0 0 0"/>
-	</xacro:rubber_wheel>
-	<xacro:rubber_wheel name="front_left" parent="base_link" reflect="1" hq="${hq}">
+	</xacro:omni_wheel>
+	<xacro:omni_wheel name="front_left" parent="base_link" reflect="true" hq="true">
 		<origin xyz="${wheel_offset_x} ${wheel_offset_y} ${wheel_offset_z}" rpy="0 0 0"/>
-	</xacro:rubber_wheel>
-	<xacro:rubber_wheel name="back_left" parent="base_link" reflect="1" hq="${hq}">
+	</xacro:omni_wheel>
+	<xacro:omni_wheel name="back_left" parent="base_link" reflect="false" hq="true">
 		<origin xyz="-${wheel_offset_x} ${wheel_offset_y} ${wheel_offset_z}" rpy="0 0 0"/>
-	</xacro:rubber_wheel>
-	<xacro:rubber_wheel name="back_right" parent="base_link" reflect="0" hq="${hq}">
+	</xacro:omni_wheel>
+	<xacro:omni_wheel name="back_right" parent="base_link" reflect="true" hq="true">
 		<origin xyz="-${wheel_offset_x} -${wheel_offset_y} ${wheel_offset_z}" rpy="0 0 0"/>
-	</xacro:rubber_wheel>
+	</xacro:omni_wheel>
 	<!-- SENSORS -->
 	<xacro:sensor_hokuyo_utm30lx name="hokuyo" parent="base_link">

File: summit_xl_description/urdf/bases/summit_xl_base.gazebo.xacro (robot description, xacro)
@@ -1,6 +1,6 @@
 <?xml version="1.0"?>
 <robot xmlns:xacro="http://ros.org/wiki/xacro">
-  <!-- ros_control skid steer plugin -->
-  <xacro:macro name="summit_xl_skid_gazebo">
+  <!-- ros control plugin -->
+  <xacro:macro name="ros_control">
     <gazebo>
       <plugin name="ros_control" filename="libgazebo_ros_control.so">
@@ -11,4 +11,7 @@
       </plugin>
     </gazebo>
+	</xacro:macro>
+	<!-- skid steering plugin -->
+	<xacro:macro name="skid_steering">
     <gazebo>
       <plugin name="skid_steer_drive_controller" filename="libgazebo_ros_skid_steer_drive.so">
@@ -31,4 +34,15 @@
     </gazebo>
   </xacro:macro>
+  <xacro:macro name="omni_steering">
+		<gazebo>
+	    <plugin name="omni_steering" filename="libgazebo_ros_planar_move.so">
+	      <commandTopic>/summit_xl/robot_control/command</commandTopic>
+	      <odometryTopic>/summit_xl/odom</odometryTopic>
+	      <odometryFrame>odom</odometryFrame>
+	      <odometryRate>20.0</odometryRate>
+	      <robotBaseFrame>base_footprint</robotBaseFrame>
+	    </plugin>
+	  </gazebo>
+  </xacro:macro>
   <gazebo reference="base_footprint">
     <material>Gazebo/Green</material>

File: summit_xl_description/urdf/wheels/omni_wheel.urdf.xacro (robot description, xacro)
@@ -4,5 +4,5 @@
   <!-- Wheels -->
   <property name="wheel_radius" value="0.117" />
-  <property name="wheel_height" value="0.12" />
+  <property name="wheel_height" value="0.14" />
   <property name="wheel_mass" value="6.5" /> <!-- in kg-->
   <macro name="cylinder_inertia" params="m r h">
@@ -33,5 +33,5 @@
               <mesh filename="package://summit_xl_description/meshes/wheels/omni_wheel_2.dae" />
             </geometry>
-		  </xacro:unless>
+					</xacro:unless>
         </xacro:if>
         <xacro:unless value="${hq}">
@@ -46,7 +46,18 @@
       </visual>
       <collision>
-		<origin xyz="0 0 0" rpy="0 0 0" />
+				<origin xyz="0 0 0" rpy="${PI/2} 0 0" />
         <geometry>
+<!--
           <sphere radius="${wheel_radius}" />
+-->
+<!--
+          <xacro:if value="${reflect}">
+              <mesh filename="package://summit_xl_description/meshes/wheels/omni_wheel_1.dae" />
+          </xacro:if>
+          <xacro:unless value="${reflect}">
+              <mesh filename="package://summit_xl_description/meshes/wheels/omni_wheel_2.dae" />
+					</xacro:unless>
+-->
+					<cylinder length="${wheel_height}" radius="${wheel_radius}" />
         </geometry>
       </collision>
@@ -72,5 +83,5 @@
 		<kd value="1.0" />
 		<fdir1 value="1 0 0"/>
-      <material>Gazebo/Gray</material>
+      <material>Gazebo/Grey</material>
       <turnGravityOff>false</turnGravityOff>
     </gazebo>

File: summit_xl_description/urdf/wheels/rubber_wheel.urdf.xacro (robot description, xacro)
@@ -4,5 +4,5 @@
   <!-- Wheels -->
   <property name="wheel_radius" value="0.117" />
-  <property name="wheel_height" value="0.12" />
+  <property name="wheel_height" value="0.14" />
   <property name="wheel_mass" value="6.5" /> <!-- in kg-->
   <xacro:macro name="cylinder_inertia" params="m r h">
