Commit message: summit_xl_description: adding fotonic component

File: summit_xl_description/robots/summit_xl.urdf.xacro (robot description, xacro)
@@ -9,4 +9,5 @@
   <xacro:include filename="$(find summit_xl_description)/urdf/sensors/kinect.urdf.xacro" />
   <xacro:include filename="$(find summit_xl_description)/urdf/sensors/hokuyo.urdf.xacro" />
+  <xacro:include filename="$(find summit_xl_description)/urdf/sensors/fotonic.urdf.xacro" />
   <!-- Robot mechanical and motor parameters -->
   <xacro:property name="PI" value="3.1415926535897931"/>
@@ -68,4 +69,7 @@
     <origin xyz="0.0 0.0 0.310" rpy="0 0 0"/>
   </hokuyo_sensor>
+  <sensor_fotonic name="fotonic" parent="base_link">
+		<origin xyz="0.275 0 0.260" rpy="0 0 0" />
+  </sensor_fotonic>
 	<gazebo>
 		<plugin name="ros_control" filename="libgazebo_ros_control.so">

Commit message: summit_xl_description: fixinf hokuyo component names

File: summit_xl_description/robots/summit_xl.urdf.xacro (robot description, xacro)
@@ -66,7 +66,7 @@
       </collision>
   </link>
-  <hokuyo_sensor name="hokuyo" parent="base_link">
+  <sensor_hokuyo name="hokuyo" parent="base_link">
     <origin xyz="0.0 0.0 0.310" rpy="0 0 0"/>
-  </hokuyo_sensor>
+  </sensor_hokuyo>
   <sensor_fotonic name="fotonic" parent="base_link">
 		<origin xyz="0.275 0 0.260" rpy="0 0 0" />

File: summit_xl_description/urdf/sensors/hokuyo.urdf.xacro (robot description, xacro)
@@ -1,6 +1,5 @@
 <?xml version="1.0"?>
 <robot name="sensor_hokuyo" xmlns:xacro="http://ros.org/wiki/xacro">
-	<xacro:property name="M_PI" value="3.1415926535897931" />
-  <xacro:macro name="hokuyo_sensor" params="name parent *origin">
+  <xacro:macro name="sensor_hokuyo" params="name parent *origin">
     <joint name="${name}_laser_joint" type="fixed">
       <!-- FRONT MOUNT -->
@@ -32,7 +31,7 @@
 		</link>
 		<!-- Kinect sensor for simulation -->
-		<kinect_sim_3dsensor/>
+		<sensor_hokuyo_gazebo/>
   </xacro:macro>
-  <xacro:macro name="hokuyo_sim_sensor">
+  <xacro:macro name="sensor_hokuyo_gazebo">
     <gazebo reference="${name}_laser_link">
 			<sensor type="ray" name="${name}_sensor">

Commit message: summit_xl_description: fixing kinect component

File: summit_xl_description/robots/summit_xl.urdf.xacro (robot description, xacro)
@@ -69,4 +69,7 @@
     <origin xyz="0.0 0.0 0.310" rpy="0 0 0"/>
   </sensor_hokuyo>
+  <sensor_kinect name="kinect" parent="base_link">
+		<origin xyz="0.5 0 0.5" rpy="0 0 0"/>
+  </sensor_kinect>
   <sensor_fotonic name="fotonic" parent="base_link">
 		<origin xyz="0.275 0 0.260" rpy="0 0 0" />

File: summit_xl_description/urdf/sensors/kinect.urdf.xacro (robot description, xacro)
@@ -32,66 +32,66 @@
       </inertial>
     </link>
-  <joint name="${name}_camera_joint" type="fixed">
-    <origin xyz="-0.031 0.0125 -0.016" rpy="0 0 0"/>
-    <parent link="${name}_camera_rgb_frame"/>
-    <child link="${name}_camera_link"/>
-  </joint>
-    <link name="${name}_camera_link">
-    <visual>
-     <origin xyz="0 0 0" rpy="0 0 ${M_PI/2}"/>
-      <geometry>
-       <mesh filename="package://summit_xl_description/meshes/sensors/kinect.dae"/>
-      </geometry>
-    </visual>
-	  <collision>
-      <origin xyz="0.0 0.0 0.0" rpy="0 0 0"/>
-	    <geometry>
-	      <box size="0.07271 0.27794 0.073"/>
-	    </geometry>
-	  </collision>
-    <inertial>
-      <mass value="0.001" />
-      <origin xyz="0 0 0" />
-      <inertia ixx="0.0001" ixy="0.0" ixz="0.0"
-               iyy="0.0001" iyz="0.0"
-               izz="0.0001" />
-    </inertial>
-  </link>
-  <!-- The fixed joints & links below are usually published by static_transformers launched by the OpenNi launch
-       files. However, for Gazebo simulation we need them, so we add them here.
-       (Hence, don't publish them additionally!) -->
-	<joint name="${name}_camera_depth_joint" type="fixed">
-	  <origin xyz="0 0.025 0" rpy="0 0 0" />
-	  <parent link="${name}_camera_rgb_frame" />
-	  <child link="${name}_camera_depth_frame" />
-	</joint>
-	<link name="${name}_camera_depth_frame">
-    <inertial>
-      <mass value="0.001" />
-      <origin xyz="0 0 0" />
-      <inertia ixx="0.0001" ixy="0.0" ixz="0.0"
-               iyy="0.0001" iyz="0.0"
-               izz="0.0001" />
-    </inertial>
-	</link>
-	<joint name="${name}_camera_depth_optical_joint" type="fixed">
-	  <origin xyz="0 0 0" rpy="${-M_PI/2} 0 ${-M_PI/2}" />
-	  <parent link="${name}_camera_depth_frame" />
-	  <child link="${name}_camera_depth_optical_frame" />
-	</joint>
-	<link name="${name}_camera_depth_optical_frame">
-    <inertial>
-      <mass value="0.001" />
-      <origin xyz="0 0 0" />
-      <inertia ixx="0.0001" ixy="0.0" ixz="0.0"
-               iyy="0.0001" iyz="0.0"
-               izz="0.0001" />
-    </inertial>
-	</link>
-	<!-- Kinect sensor for simulation -->
-	<kinect_sim_3dsensor/>
+	  <joint name="${name}_camera_joint" type="fixed">
+	    <origin xyz="-0.031 0.0125 -0.016" rpy="0 0 0"/>
+	    <parent link="${name}_camera_rgb_frame"/>
+	    <child link="${name}_camera_link"/>
+	  </joint>
+	    <link name="${name}_camera_link">
+	    <visual>
+	     <origin xyz="0 0 0" rpy="0 0 ${M_PI/2}"/>
+	      <geometry>
+	       <mesh filename="package://summit_xl_description/meshes/sensors/kinect.dae"/>
+	      </geometry>
+	    </visual>
+		  <collision>
+	      <origin xyz="0.0 0.0 0.0" rpy="0 0 0"/>
+		    <geometry>
+		      <box size="0.07271 0.27794 0.073"/>
+		    </geometry>
+		  </collision>
+	    <inertial>
+	      <mass value="0.001" />
+	      <origin xyz="0 0 0" />
+	      <inertia ixx="0.0001" ixy="0.0" ixz="0.0"
+	               iyy="0.0001" iyz="0.0"
+	               izz="0.0001" />
+	    </inertial>
+	  </link>
+	  <!-- The fixed joints & links below are usually published by static_transformers launched by the OpenNi launch
+	       files. However, for Gazebo simulation we need them, so we add them here.
+	       (Hence, don't publish them additionally!) -->
+		<joint name="${name}_camera_depth_joint" type="fixed">
+		  <origin xyz="0 0.025 0" rpy="0 0 0" />
+		  <parent link="${name}_camera_rgb_frame" />
+		  <child link="${name}_camera_depth_frame" />
+		</joint>
+		<link name="${name}_camera_depth_frame">
+	    <inertial>
+	      <mass value="0.001" />
+	      <origin xyz="0 0 0" />
+	      <inertia ixx="0.0001" ixy="0.0" ixz="0.0"
+	               iyy="0.0001" iyz="0.0"
+	               izz="0.0001" />
+	    </inertial>
+		</link>
+		<joint name="${name}_camera_depth_optical_joint" type="fixed">
+		  <origin xyz="0 0 0" rpy="${-M_PI/2} 0 ${-M_PI/2}" />
+		  <parent link="${name}_camera_depth_frame" />
+		  <child link="${name}_camera_depth_optical_frame" />
+		</joint>
+		<link name="${name}_camera_depth_optical_frame">
+	    <inertial>
+	      <mass value="0.001" />
+	      <origin xyz="0 0 0" />
+	      <inertia ixx="0.0001" ixy="0.0" ixz="0.0"
+	               iyy="0.0001" iyz="0.0"
+	               izz="0.0001" />
+	    </inertial>
+		</link>
+		<!-- Kinect sensor for simulation -->
+	  <sensor_kinect_gazebo/>
   </xacro:macro>
-  	<xacro:macro name="kinect_sim_3dsensor">
-    <gazebo reference="camera_link">
+  <xacro:macro name="sensor_kinect_gazebo">
+    <gazebo reference="${name}_camera_depth_frame">
       <sensor type="depth" name="camera">
         <always_on>true</always_on>

Commit message: summit_xl_description: adding axis camera component

File: summit_xl_description/robots/summit_xl.urdf.xacro (robot description, xacro)
@@ -10,4 +10,5 @@
   <xacro:include filename="$(find summit_xl_description)/urdf/sensors/hokuyo.urdf.xacro" />
   <xacro:include filename="$(find summit_xl_description)/urdf/sensors/fotonic.urdf.xacro" />
+  <xacro:include filename="$(find summit_xl_description)/urdf/sensors/axis.urdf.xacro" />
   <!-- Robot mechanical and motor parameters -->
   <xacro:property name="PI" value="3.1415926535897931"/>
@@ -20,9 +21,4 @@
   <xacro:property name="wheel_joint_velocity_limit" value="100.0" />
   <xacro:property name="wheel_mechanical_reduction" value="1.0" />
-  <xacro:property name="ptz_joint_effort_limit" value="100.0" />
-  <xacro:property name="ptz_joint_velocity_limit" value="100.0"/>
-  <xacro:property name="ptz_joint_friction" value="0.1" />
-  <xacro:property name="ptz_joint_damping" value="0.1" />
-  <xacro:property name="ptz_mechanical_reduction" value="1.0" />
   <xacro:property name="rubber_wheels" value="true" />
   <summit_xl_base name="summit_xl" />
@@ -66,13 +62,20 @@
       </collision>
   </link>
+<!--
   <sensor_hokuyo name="hokuyo" parent="base_link">
     <origin xyz="0.0 0.0 0.310" rpy="0 0 0"/>
   </sensor_hokuyo>
+-->
+<!--
   <sensor_kinect name="kinect" parent="base_link">
 		<origin xyz="0.5 0 0.5" rpy="0 0 0"/>
   </sensor_kinect>
+-->
   <sensor_fotonic name="fotonic" parent="base_link">
 		<origin xyz="0.275 0 0.260" rpy="0 0 0" />
   </sensor_fotonic>
+  <sensor_axis name="axis" parent="base_link">
+		<origin xyz="0 0 0.2825" rpy="0 0 0"/>
+  </sensor_axis>
 	<gazebo>
 		<plugin name="ros_control" filename="libgazebo_ros_control.so">

Commit message: summit_xl_description: adding gazebo common files

File: summit_xl_description/robots/summit_xl.urdf.xacro (robot description, xacro)
@@ -2,7 +2,5 @@
 <robot name="summit_xl" xmlns:xacro="http://www.ros.org/wiki/xacro">
   <!-- Import all Gazebo-customization elements, including Gazebo colors -->
-<!--
-  <xacro:include filename="$(find summit_xl_description)/urdf/summit_xl_hq.gazebo" />
--->
+	<xacro:include filename="$(find summit_xl_description)/gazebo/gazebo_skid_steering.urdf.xacro" />
   <xacro:include filename="$(find summit_xl_description)/urdf/bases/summit_xl_base.urdf.xacro" />
   <xacro:include filename="$(find summit_xl_description)/urdf/wheels/rubber_wheel.urdf.xacro" />
@@ -38,5 +36,5 @@
   <!-- IMU SENSOR -->
   <joint name="imu_joint" type="fixed">
-      <axis xyz="1 0 0"/> <!-- 0 1 0 -->
+      <axis xyz="1 0 0"/>
       <origin xyz="0 0 0.2825"/>
       <parent link="base_link"/>
@@ -78,29 +76,3 @@
 		<origin xyz="0 0 0.2825" rpy="0 0 0"/>
   </sensor_axis>
-	<gazebo>
-		<plugin name="ros_control" filename="libgazebo_ros_control.so">
-			 <robotNamespace>$(arg namespace)</robotNamespace>
-			 <controlPeriod>0.003</controlPeriod>
-     <robotSimType>gazebo_ros_control/DefaultRobotHWSim</robotSimType>
-		</plugin>
-	</gazebo>
-	<gazebo>
-		<plugin name="skid_steer_drive_controllerasdasdasd" filename="libgazebo_ros_skid_steer_drive.so">
-  	  <robotNamespace>$(arg namespace)</robotNamespace>
-      <updateRate>100.0</updateRate>
-      <leftFrontJoint>joint_front_left_wheel</leftFrontJoint>
-      <rightFrontJoint>joint_front_right_wheel</rightFrontJoint>
-      <leftRearJoint>joint_back_left_wheel</leftRearJoint>
-      <rightRearJoint>joint_back_right_wheel</rightRearJoint>
-      <wheelSeparation>0.308</wheelSeparation>
-      <wheelDiameter>0.125</wheelDiameter>
-      <robotBaseFrame>$(arg namespace)/base_footprint</robotBaseFrame>
-      <torque>25</torque>
-      <topicName>cmd_vel</topicName>
-      <commandTopic>summit_xl_steer_drive_controller/command</commandTopic>
-      <odometryTopic>odom</odometryTopic>
-      <odometryFrame>$(arg namespace)/odom</odometryFrame>
-      <broadcastTF>1</broadcastTF>
-		</plugin>
-	</gazebo>
 </robot>

File: summit_xl_description/urdf/bases/summit_xl_base.urdf.xacro (robot description, xacro)
@@ -1,6 +1,4 @@
 <?xml version="1.0"?>
 <robot name="summit_xl" xmlns:xacro="http://www.ros.org/wiki/xacro">
-  <!-- Import all Gazebo-customization elements, including Gazebo colors -->
-  <xacro:include filename="$(find summit_xl_description)/urdf/summit_xl.gazebo"/>
   <xacro:macro name="summit_xl_base" params="name">
   <!-- Robot mechanical and motor parameters -->
@@ -20,4 +18,10 @@
   <xacro:property name="ptz_joint_damping" value="0.1" />
   <xacro:property name="ptz_mechanical_reduction" value="1.0" />
+	<gazebo reference="base_footprint">
+    <material>Gazebo/Green</material>
+  </gazebo>
+  <gazebo reference="base_link">
+    <material>Gazebo/Red</material>
+  </gazebo>
   <!-- BASE FOOTPRINT -->
   <!-- base_footprint is a fictitious link(frame) that is on the ground right below base_link origin,

File: summit_xl_description/urdf/wheels/rubber_wheel.urdf.xacro (robot description, xacro)
@@ -67,10 +67,10 @@
     </transmission>
     <gazebo reference="${name}_wheel">
-		<mu1 value="5.0"/>
-		<mu2 value="0.5"/>
-		<kp value="10000000.0" />
-		<kd value="1.0" />
-		<fdir1 value="1 0 0"/>
-      <material>Gazebo/Gray</material>
+			<mu1 value="5.0"/>
+			<mu2 value="0.5"/>
+			<kp value="10000000.0" />
+			<kd value="1.0" />
+			<fdir1 value="1 0 0"/>
+      <material>Gazebo/Grey</material>
       <turnGravityOff>false</turnGravityOff>
     </gazebo>

Commit message: deleting summit_xl_hq version, default summit_xl will be hq

File: summit_xl_description/robots/summit_xl.urdf.xacro (robot description, xacro)
@@ -2,77 +2,47 @@
 <robot name="summit_xl" xmlns:xacro="http://www.ros.org/wiki/xacro">
   <!-- Import all Gazebo-customization elements, including Gazebo colors -->
-	<xacro:include filename="$(find summit_xl_description)/gazebo/gazebo_skid_steering.urdf.xacro" />
+  <xacro:include filename="$(find summit_xl_description)/urdf/bases/summit_xl_base.gazebo.xacro" />
   <xacro:include filename="$(find summit_xl_description)/urdf/bases/summit_xl_base.urdf.xacro" />
   <xacro:include filename="$(find summit_xl_description)/urdf/wheels/rubber_wheel.urdf.xacro" />
-  <xacro:include filename="$(find summit_xl_description)/urdf/sensors/kinect.urdf.xacro" />
-  <xacro:include filename="$(find summit_xl_description)/urdf/sensors/hokuyo.urdf.xacro" />
-  <xacro:include filename="$(find summit_xl_description)/urdf/sensors/fotonic.urdf.xacro" />
+  <xacro:include filename="$(find summit_xl_description)/urdf/sensors/hokuyo_urg04lx.urdf.xacro" />
+  <xacro:include filename="$(find summit_xl_description)/urdf/sensors/hokuyo_utm30lx.urdf.xacro" />
   <xacro:include filename="$(find summit_xl_description)/urdf/sensors/axis.urdf.xacro" />
+  <xacro:include filename="$(find summit_xl_description)/urdf/sensors/imu.urdf.xacro" />
   <!-- Robot mechanical and motor parameters -->
   <xacro:property name="PI" value="3.1415926535897931"/>
-  <xacro:property name="wheel_offset_x" value="0.223" />    <!-- x,y,z in base_link CS -->
-  <xacro:property name="wheel_offset_y" value="0.234" />
+  <xacro:property name="wheel_offset_x" value="0.229" />    <!-- x,y,z in base_link CS -->
+  <xacro:property name="wheel_offset_y" value="0.234" />    <!-- y distance between base_link and the center of the wheel -->
   <xacro:property name="wheel_offset_z" value="0.0" />
-  <xacro:property name="wheel_joint_damping" value="0.0" />
-  <xacro:property name="wheel_joint_friction" value="0.0" />
-  <xacro:property name="wheel_joint_effort_limit" value="100.0" />
-  <xacro:property name="wheel_joint_velocity_limit" value="100.0" />
-  <xacro:property name="wheel_mechanical_reduction" value="1.0" />
-  <xacro:property name="rubber_wheels" value="true" />
-  <summit_xl_base name="summit_xl" />
-    <!-- WHEELS -->
-  <rubber_wheel name="front_right" parent="base_link" reflect="0">
+	<!-- Flag to select the high or low quality model -->
+  <xacro:property name="hq" value="true" />
+  <xacro:summit_xl_base name="summit_xl" publish_bf="true" hq="${hq}" />
+  <xacro:summit_xl_skid_gazebo/>
+  <!-- WHEELS -->
+  <xacro:rubber_wheel name="front_right" parent="base_link" reflect="0" hq="${hq}">
     <origin xyz="${wheel_offset_x} -${wheel_offset_y} ${wheel_offset_z}" rpy="0 0 0"/>
-  </rubber_wheel>
-  <rubber_wheel name="front_left" parent="base_link" reflect="1">
+  </xacro:rubber_wheel>
+  <xacro:rubber_wheel name="front_left" parent="base_link" reflect="1" hq="${hq}">
     <origin xyz="${wheel_offset_x} ${wheel_offset_y} ${wheel_offset_z}" rpy="0 0 0"/>
-  </rubber_wheel>
-  <rubber_wheel name="back_left" parent="base_link" reflect="1">
+  </xacro:rubber_wheel>
+  <xacro:rubber_wheel name="back_left" parent="base_link" reflect="1" hq="${hq}">
     <origin xyz="-${wheel_offset_x} ${wheel_offset_y} ${wheel_offset_z}" rpy="0 0 0"/>
-  </rubber_wheel>
-  <rubber_wheel name="back_right" parent="base_link" reflect="0">
+  </xacro:rubber_wheel>
+  <xacro:rubber_wheel name="back_right" parent="base_link" reflect="0" hq="${hq}">
     <origin xyz="-${wheel_offset_x} -${wheel_offset_y} ${wheel_offset_z}" rpy="0 0 0"/>
-  </rubber_wheel>
-  <!-- IMU SENSOR -->
-  <joint name="imu_joint" type="fixed">
-      <axis xyz="1 0 0"/>
-      <origin xyz="0 0 0.2825"/>
-      <parent link="base_link"/>
-      <child link="imu_link"/>
-  </joint>
-  <link name="imu_link">
-      <inertial>
-        <mass value="0.001"/>
-        <origin rpy="0 0 0" xyz="0 0 0"/>
-        <inertia ixx="0.0001" ixy="0" ixz="0" iyy="0.000001" iyz="0" izz="0.0001"/>
-      </inertial>
-      <visual>
-        <origin rpy="0 0 0" xyz="0 0 0"/>
-        <geometry>
-          <box size="0.001 0.001 0.001"/>
-        </geometry>
-      </visual>
-      <collision>
-        <origin rpy="0 0 0" xyz="0 0 0"/>
-        <geometry>
-          <box size=".001 .001 .001"/>
-        </geometry>
-      </collision>
-  </link>
+  </xacro:rubber_wheel>
+	<!-- SENSORS -->
+  <xacro:sensor_hokuyo_utm30lx name="hokuyo" parent="base_link">
+    <origin xyz="0.0 0.0 0.33" rpy="0 0 0"/>
+  </xacro:sensor_hokuyo_utm30lx>
 <!--
-  <sensor_hokuyo name="hokuyo" parent="base_link">
-    <origin xyz="0.0 0.0 0.310" rpy="0 0 0"/>
-  </sensor_hokuyo>
+  <xacro:sensor_hokuyo_urg04lx name="hokuyo1" parent="base_link">
+    <origin xyz="0.0 0.0 0.36" rpy="0 0 0"/>
+  </xacro:sensor_hokuyo_urg04lx>
 -->
-<!--
-  <sensor_kinect name="kinect" parent="base_link">
-		<origin xyz="0.5 0 0.5" rpy="0 0 0"/>
-  </sensor_kinect>
--->
-  <sensor_fotonic name="fotonic" parent="base_link">
-		<origin xyz="0.275 0 0.260" rpy="0 0 0" />
-  </sensor_fotonic>
-  <sensor_axis name="axis" parent="base_link">
-		<origin xyz="0 0 0.2825" rpy="0 0 0"/>
-  </sensor_axis>
+  <xacro:sensor_axis name="camera" parent="base_link">
+		<origin xyz="0.19 0 0.17" rpy="0 ${15*PI/180} 0"/>
+  </xacro:sensor_axis>
+  <xacro:sensor_imu name="imu" parent="base_link">
+		<origin xyz="-0.18 0.0 0.170" rpy="0 0 0"/>
+  </xacro:sensor_imu>
 </robot>

Commit message: summit_xl_description: adding gps sensor

File: summit_xl_description/robots/summit_xl.urdf.xacro (robot description, xacro)
@@ -9,4 +9,5 @@
   <xacro:include filename="$(find summit_xl_description)/urdf/sensors/axis.urdf.xacro" />
   <xacro:include filename="$(find summit_xl_description)/urdf/sensors/imu.urdf.xacro" />
+  <xacro:include filename="$(find summit_xl_description)/urdf/sensors/gps.urdf.xacro" />
   <!-- Robot mechanical and motor parameters -->
   <xacro:property name="PI" value="3.1415926535897931"/>
@@ -46,3 +47,6 @@
 		<origin xyz="-0.18 0.0 0.170" rpy="0 0 0"/>
   </xacro:sensor_imu>
+  <xacro:sensor_gps name="gps" parent="base_link">
+		<origin xyz="-0.22 0 0.275" rpy="0 0 0"/>
+	</xacro:sensor_gps>
 </robot>

Commit message: summit_xl_description: adding a file with all sensors and commenting summit_xl.urdf.xacro

File: summit_xl_description/robots/summit_xl.urdf.xacro (robot description, xacro)
@@ -1,21 +1,27 @@
 <?xml version="1.0"?>
 <robot name="summit_xl" xmlns:xacro="http://www.ros.org/wiki/xacro">
-  <!-- Import all Gazebo-customization elements, including Gazebo colors -->
-  <xacro:include filename="$(find summit_xl_description)/urdf/bases/summit_xl_base.gazebo.xacro" />
+	<!-- First we import all posible elements defined in the urdf.xacro files. All these elements are defined as macro:xacros -->
+	<!-------------------------------------------------------------------------------------------------------------------------->
+  <!-- Import summit XL base elements -->
   <xacro:include filename="$(find summit_xl_description)/urdf/bases/summit_xl_base.urdf.xacro" />
+  <!-- Import summit XL wheels -->
   <xacro:include filename="$(find summit_xl_description)/urdf/wheels/rubber_wheel.urdf.xacro" />
-  <xacro:include filename="$(find summit_xl_description)/urdf/sensors/hokuyo_urg04lx.urdf.xacro" />
-  <xacro:include filename="$(find summit_xl_description)/urdf/sensors/hokuyo_utm30lx.urdf.xacro" />
-  <xacro:include filename="$(find summit_xl_description)/urdf/sensors/axis.urdf.xacro" />
-  <xacro:include filename="$(find summit_xl_description)/urdf/sensors/imu.urdf.xacro" />
-  <xacro:include filename="$(find summit_xl_description)/urdf/sensors/gps.urdf.xacro" />
-  <!-- Robot mechanical and motor parameters -->
+  <!-- Import all available sensors -->
+  <xacro:include filename="$(find summit_xl_description)/urdf/sensors/all_sensors.urdf.xacro" />
+  <!-- Global parameters -->
+  <!----------------------->
   <xacro:property name="PI" value="3.1415926535897931"/>
-  <xacro:property name="wheel_offset_x" value="0.229" />    <!-- x,y,z in base_link CS -->
-  <xacro:property name="wheel_offset_y" value="0.234" />    <!-- y distance between base_link and the center of the wheel -->
+  <!-- Wheel parameters -->
+  <xacro:property name="wheel_offset_x" value="0.229" />    <!-- x,y,z in translation from base_link to the center of the wheel -->
+  <xacro:property name="wheel_offset_y" value="0.234" />
   <xacro:property name="wheel_offset_z" value="0.0" />
 	<!-- Flag to select the high or low quality model -->
   <xacro:property name="hq" value="true" />
+	<!-- Elements -->
+	<!-------------->
+	<!-- Here we create the robot elements using the xacro:macros imported at the beggining of this file -->
+	<!-- Summit XL base -->
   <xacro:summit_xl_base name="summit_xl" publish_bf="true" hq="${hq}" />
+  <!-- Summit XL movement pluggins -->
   <xacro:summit_xl_skid_gazebo/>
   <!-- WHEELS -->
@@ -38,5 +44,5 @@
 <!--
   <xacro:sensor_hokuyo_urg04lx name="hokuyo1" parent="base_link">
-    <origin xyz="0.0 0.0 0.36" rpy="0 0 0"/>
+    <origin xyz="-0.1 0.0 0.33" rpy="0 0 0"/>
   </xacro:sensor_hokuyo_urg04lx>
 -->

File: summit_xl_description/urdf/bases/summit_xl_base.urdf.xacro (robot description, xacro)
@@ -1,4 +1,5 @@
 <?xml version="1.0"?>
 <robot name="summit_xl" xmlns:xacro="http://www.ros.org/wiki/xacro">
+	<xacro:include filename="$(find summit_xl_description)/urdf/bases/summit_xl_base.gazebo.xacro" />
   <xacro:macro name="summit_xl_base" params="name publish_bf hq">
   <!-- Robot mechanical and motor parameters -->
