Commit message: summit_xl_description: fixing kinect sensor

File: summit_xl_description/robots/summit_xl.urdf.xacro (robot description, xacro)
@@ -60,3 +60,8 @@
 		<origin xyz="-0.22 0 0.275" rpy="0 0 0"/>
 	</xacro:sensor_gps>
+<!--
+  <xacro:sensor_kinect name="kinect" parent="base_link">
+    <origin xyz="0.3 0.0 0.16" rpy="0 0 0"/>
+  </xacro:sensor_kinect>
+-->
 </robot>

File: summit_xl_description/urdf/sensors/all_sensors.urdf.xacro (robot description, xacro)
@@ -2,13 +2,17 @@
 <robot name="all_sensors" xmlns:xacro="http://ros.org/wiki/xacro">
 	<!-- This file unifies all sensors that can be used on simulation, defined as xacro:macros -->
+  <!-- Axis p5512 -->
+  <xacro:include filename="$(find summit_xl_description)/urdf/sensors/axis.urdf.xacro" />
+	<!-- Fotonic -->
+  <xacro:include filename="$(find summit_xl_description)/urdf/sensors/fotonic.urdf.xacro" />
+	<!-- GPS -->
+  <xacro:include filename="$(find summit_xl_description)/urdf/sensors/gps.urdf.xacro" />
 	<!-- Hokuyo urg04lx -->
 	<xacro:include filename="$(find summit_xl_description)/urdf/sensors/hokuyo_urg04lx.urdf.xacro" />
 	<!-- Hokuyo utm30lx -->
   <xacro:include filename="$(find summit_xl_description)/urdf/sensors/hokuyo_utm30lx.urdf.xacro" />
-  <!-- Axis p5512 -->
-  <xacro:include filename="$(find summit_xl_description)/urdf/sensors/axis.urdf.xacro" />
   <!-- Imu -->
   <xacro:include filename="$(find summit_xl_description)/urdf/sensors/imu.urdf.xacro" />
-  <!-- GPS -->
-  <xacro:include filename="$(find summit_xl_description)/urdf/sensors/gps.urdf.xacro" />
+  <!-- Kinect -->
+  <xacro:include filename="$(find summit_xl_description)/urdf/sensors/kinect.urdf.xacro" />
 </robot>

File: summit_xl_description/urdf/sensors/kinect.urdf.xacro (robot description, xacro)
@@ -3,38 +3,10 @@
   <xacro:property name="M_PI" value="3.1415926535897931" />
   <xacro:macro name="sensor_kinect" params="name parent *origin">
-    <joint name="${name}_camera_rgb_joint" type="fixed">
-      <insert_block name="origin" />
-      <parent link="${parent}"/>
-      <child link="${name}_camera_rgb_frame" />
-    </joint>
-    <link name="${name}_camera_rgb_frame">
-      <inertial>
-        <mass value="0.001" />
-        <origin xyz="0 0 0" />
-        <inertia ixx="0.0001" ixy="0.0" ixz="0.0"
-                 iyy="0.0001" iyz="0.0"
-                 izz="0.0001" />
-      </inertial>
-    </link>
-    <joint name="${name}_camera_rgb_optical_joint" type="fixed">
-      <origin xyz="0 0 0" rpy="${-M_PI/2} 0 ${-M_PI/2}" />
-      <parent link="${name}_camera_rgb_frame" />
-      <child link="${name}_camera_rgb_optical_frame" />
-    </joint>
-    <link name="${name}_camera_rgb_optical_frame">
-      <inertial>
-        <mass value="0.001" />
-        <origin xyz="0 0 0" />
-        <inertia ixx="0.0001" ixy="0.0" ixz="0.0"
-                 iyy="0.0001" iyz="0.0"
-                 izz="0.0001" />
-      </inertial>
-    </link>
-	  <joint name="${name}_camera_joint" type="fixed">
-	    <origin xyz="-0.031 0.0125 -0.016" rpy="0 0 0"/>
-	    <parent link="${name}_camera_rgb_frame"/>
-	    <child link="${name}_camera_link"/>
+    <joint name="${name}_cam_joint" type="fixed">
+	    <insert_block name="origin" />
+	    <parent link="${parent}"/>
+	    <child link="${name}_cam_link"/>
 	  </joint>
-	    <link name="${name}_camera_link">
+	  <link name="${name}_cam_link">
 	    <visual>
 	     <origin xyz="0 0 0" rpy="0 0 ${M_PI/2}"/>
@@ -57,13 +29,41 @@
 	    </inertial>
 	  </link>
+    <joint name="${name}_cam_rgb_joint" type="fixed">
+      <origin xyz="0.031 -0.0125 0.016" rpy="0 0 0"/>
+      <parent link="${name}_cam_link"/>
+      <child link="${name}_cam_rgb_frame" />
+    </joint>
+    <link name="${name}_cam_rgb_frame">
+      <inertial>
+        <mass value="0.001" />
+        <origin xyz="0 0 0" />
+        <inertia ixx="0.0001" ixy="0.0" ixz="0.0"
+                 iyy="0.0001" iyz="0.0"
+                 izz="0.0001" />
+      </inertial>
+    </link>
+    <joint name="${name}_cam_rgb_optical_joint" type="fixed">
+      <origin xyz="0 0 0" rpy="${-M_PI/2} 0 ${-M_PI/2}" />
+      <parent link="${name}_cam_rgb_frame" />
+      <child link="${name}_cam_rgb_optical_frame" />
+    </joint>
+    <link name="${name}_cam_rgb_optical_frame">
+      <inertial>
+        <mass value="0.001" />
+        <origin xyz="0 0 0" />
+        <inertia ixx="0.0001" ixy="0.0" ixz="0.0"
+                 iyy="0.0001" iyz="0.0"
+                 izz="0.0001" />
+      </inertial>
+    </link>
 	  <!-- The fixed joints & links below are usually published by static_transformers launched by the OpenNi launch
 	       files. However, for Gazebo simulation we need them, so we add them here.
 	       (Hence, don't publish them additionally!) -->
-		<joint name="${name}_camera_depth_joint" type="fixed">
+		<joint name="${name}_cam_depth_joint" type="fixed">
 		  <origin xyz="0 0.025 0" rpy="0 0 0" />
-		  <parent link="${name}_camera_rgb_frame" />
-		  <child link="${name}_camera_depth_frame" />
+		  <parent link="${name}_cam_rgb_frame" />
+		  <child link="${name}_cam_depth_frame" />
 		</joint>
-		<link name="${name}_camera_depth_frame">
+		<link name="${name}_cam_depth_frame">
 	    <inertial>
 	      <mass value="0.001" />
@@ -74,10 +74,10 @@
 	    </inertial>
 		</link>
-		<joint name="${name}_camera_depth_optical_joint" type="fixed">
+		<joint name="${name}_cam_depth_optical_joint" type="fixed">
 		  <origin xyz="0 0 0" rpy="${-M_PI/2} 0 ${-M_PI/2}" />
-		  <parent link="${name}_camera_depth_frame" />
-		  <child link="${name}_camera_depth_optical_frame" />
+		  <parent link="${name}_cam_depth_frame" />
+		  <child link="${name}_cam_depth_optical_frame" />
 		</joint>
-		<link name="${name}_camera_depth_optical_frame">
+		<link name="${name}_cam_depth_optical_frame">
 	    <inertial>
 	      <mass value="0.001" />
@@ -91,12 +91,7 @@
 	  <sensor_kinect_gazebo/>
   </xacro:macro>
-<<<<<<< HEAD
-  	<xacro:macro name="kinect_sim_3dsensor">
-    <gazebo reference="${name}_camera_link">
-=======
   <xacro:macro name="sensor_kinect_gazebo">
-    <gazebo reference="${name}_camera_depth_frame">
->>>>>>> 3458c358f882804e39b6f09caff537bf7e09d839
-      <sensor type="depth" name="camera">
+    <gazebo reference="${name}_cam_depth_frame">
+      <sensor type="depth" name="cam">
         <always_on>true</always_on>
         <update_rate>20.0</update_rate>
@@ -113,5 +108,5 @@
           </clip>
         </camera>
-        <plugin name="kinect_camera_controller" filename="libgazebo_ros_openni_kinect.so">
+        <plugin name="kinect_cam_controller" filename="libgazebo_ros_openni_kinect.so">
           <cameraName>${name}</cameraName>
           <alwaysOn>true</alwaysOn>
@@ -122,5 +117,5 @@
           <cameraInfoTopicName>rgb/camera_info</cameraInfoTopicName>
           <depthImageCameraInfoTopicName>depth/camera_info</depthImageCameraInfoTopicName>
-          <frameName>${name}_camera_depth_optical_frame</frameName>
+          <frameName>${name}_cam_depth_optical_frame</frameName>
           <baseline>0.1</baseline>
           <distortion_k1>0.0</distortion_k1>

Commit message: summit_xl_description: fixing fotonic model

File: summit_xl_description/robots/summit_xl.urdf.xacro (robot description, xacro)
@@ -65,3 +65,8 @@
   </xacro:sensor_kinect>
 -->
+<!--
+  <xacro:sensor_fotonic name="fotonic" parent="base_link">
+    <origin xyz="0.3 0.0 0.24" rpy="0 0 0"/>
+  </xacro:sensor_fotonic>
+-->
 </robot>

File: summit_xl_description/urdf/sensors/fotonic.urdf.xacro (robot description, xacro)
@@ -18,6 +18,9 @@
 	    <visual>
 	      <origin xyz="-0.275 0 -0.260" rpy="0 0 0" /> <!-- to center the .dae model -->
+	      <material name="fotonic_color">
+           <color rgba="0.5 0.5 0.5 1"/>
+        </material>
 	      <geometry>
-					<mesh filename= "package://summit_xl_description/meshes/xl_fotonic/fotonic.dae" scale="1.0 1.0 1.0"/>
+					<mesh filename= "package://summit_xl_description/meshes/xl_fotonic/fotonic.stl" scale="1.0 1.0 1.0"/>
 	      </geometry>
 	    </visual>
@@ -25,5 +28,5 @@
 	      <origin xyz="-0.275 0 -0.260" rpy="0 0 0" />
 	      <geometry>
-	        <mesh filename= "package://summit_xl_description/meshes/xl_fotonic/fotonic.dae" scale="1.0 1.0 1.0"/>
+	        <mesh filename= "package://summit_xl_description/meshes/xl_fotonic/fotonic.stl" scale="1.0 1.0 1.0"/>
 	      </geometry>
 	    </collision>
@@ -61,4 +64,7 @@
   </xacro:macro>
   <xacro:macro name="sensor_fotonic_gazebo">
+		<gazebo reference="${name}_link">
+      <material>Gazebo/Grey</material>
+    </gazebo>
     <gazebo reference="${name}_depth_frame">
 	    <sensor type="depth" name="fotonic">

Commit message: Update summit_xl.urdf.xacro
Fixing tab errors

File: summit_xl_description/robots/summit_xl.urdf.xacro (robot description, xacro)
@@ -5,20 +5,20 @@
 	<!-- ***************** -->
 	<!-- First we import all posible elements defined in the urdf.xacro files. All these elements are defined as macro:xacros -->
-  <!-- Import summit XL base elements -->
-  <xacro:include filename="$(find summit_xl_description)/urdf/bases/summit_xl_base.urdf.xacro" />
-  <!-- Import summit XL wheels -->
-  <xacro:include filename="$(find summit_xl_description)/urdf/wheels/rubber_wheel.urdf.xacro" />
-  <!-- Import all available sensors -->
-  <xacro:include filename="$(find summit_xl_description)/urdf/sensors/all_sensors.urdf.xacro" />
+	<!-- Import summit XL base elements -->
+	<xacro:include filename="$(find summit_xl_description)/urdf/bases/summit_xl_base.urdf.xacro" />
+	<!-- Import summit XL wheels -->
+	<xacro:include filename="$(find summit_xl_description)/urdf/wheels/rubber_wheel.urdf.xacro" />
+	<!-- Import all available sensors -->
+	<xacro:include filename="$(find summit_xl_description)/urdf/sensors/all_sensors.urdf.xacro" />
 	<!-- ***************** -->
-  <!-- Global parameters -->
+	<!-- Global parameters -->
 	<!-- ***************** -->
-  <xacro:property name="PI" value="3.1415926535897931"/>
-  <!-- Wheel parameters -->
-  <xacro:property name="wheel_offset_x" value="0.229" />    <!-- x,y,z in translation from base_link to the center of the wheel -->
-  <xacro:property name="wheel_offset_y" value="0.234" />
-  <xacro:property name="wheel_offset_z" value="0.0" />
+	<xacro:property name="PI" value="3.1415926535897931"/>
+	<!-- Wheel parameters -->
+	<xacro:property name="wheel_offset_x" value="0.229" />    <!-- x,y,z in translation from base_link to the center of the wheel -->
+	<xacro:property name="wheel_offset_y" value="0.234" />
+	<xacro:property name="wheel_offset_z" value="0.0" />
 	<!-- Flag to select the high or low quality model -->
-  <xacro:property name="hq" value="true" />
+	<xacro:property name="hq" value="true" />
 	<!-- *************** -->
 	<!-- Robots Elements -->
@@ -26,47 +26,47 @@
 	<!-- Here we create the robot elements using the xacro:macros imported at the beggining of this file -->
 	<!-- Summit XL base -->
-  <xacro:summit_xl_base name="summit_xl" publish_bf="true" hq="${hq}" />
-  <!-- Summit XL movement pluggins -->
-  <xacro:summit_xl_skid_gazebo/>
-  <!-- WHEELS -->
-  <xacro:rubber_wheel name="front_right" parent="base_link" reflect="0" hq="${hq}">
-    <origin xyz="${wheel_offset_x} -${wheel_offset_y} ${wheel_offset_z}" rpy="0 0 0"/>
-  </xacro:rubber_wheel>
-  <xacro:rubber_wheel name="front_left" parent="base_link" reflect="1" hq="${hq}">
-    <origin xyz="${wheel_offset_x} ${wheel_offset_y} ${wheel_offset_z}" rpy="0 0 0"/>
-  </xacro:rubber_wheel>
-  <xacro:rubber_wheel name="back_left" parent="base_link" reflect="1" hq="${hq}">
-    <origin xyz="-${wheel_offset_x} ${wheel_offset_y} ${wheel_offset_z}" rpy="0 0 0"/>
-  </xacro:rubber_wheel>
-  <xacro:rubber_wheel name="back_right" parent="base_link" reflect="0" hq="${hq}">
-    <origin xyz="-${wheel_offset_x} -${wheel_offset_y} ${wheel_offset_z}" rpy="0 0 0"/>
-  </xacro:rubber_wheel>
+	<xacro:summit_xl_base name="summit_xl" publish_bf="true" hq="${hq}" />
+	<!-- Summit XL movement pluggins -->
+	<xacro:summit_xl_skid_gazebo/>
+	<!-- WHEELS -->
+	<xacro:rubber_wheel name="front_right" parent="base_link" reflect="0" hq="${hq}">
+		<origin xyz="${wheel_offset_x} -${wheel_offset_y} ${wheel_offset_z}" rpy="0 0 0"/>
+	</xacro:rubber_wheel>
+	<xacro:rubber_wheel name="front_left" parent="base_link" reflect="1" hq="${hq}">
+		<origin xyz="${wheel_offset_x} ${wheel_offset_y} ${wheel_offset_z}" rpy="0 0 0"/>
+	</xacro:rubber_wheel>
+	<xacro:rubber_wheel name="back_left" parent="base_link" reflect="1" hq="${hq}">
+		<origin xyz="-${wheel_offset_x} ${wheel_offset_y} ${wheel_offset_z}" rpy="0 0 0"/>
+	</xacro:rubber_wheel>
+	<xacro:rubber_wheel name="back_right" parent="base_link" reflect="0" hq="${hq}">
+		<origin xyz="-${wheel_offset_x} -${wheel_offset_y} ${wheel_offset_z}" rpy="0 0 0"/>
+	</xacro:rubber_wheel>
 	<!-- SENSORS -->
-  <xacro:sensor_hokuyo_utm30lx name="hokuyo" parent="base_link">
-    <origin xyz="0.0 0.0 0.33" rpy="0 0 0"/>
-  </xacro:sensor_hokuyo_utm30lx>
+	<xacro:sensor_hokuyo_utm30lx name="hokuyo" parent="base_link">
+		<origin xyz="0.0 0.0 0.33" rpy="0 0 0"/>
+	</xacro:sensor_hokuyo_utm30lx>
 <!--
-  <xacro:sensor_hokuyo_urg04lx name="hokuyo1" parent="base_link">
-    <origin xyz="-0.1 0.0 0.33" rpy="0 0 0"/>
-  </xacro:sensor_hokuyo_urg04lx>
+	<xacro:sensor_hokuyo_urg04lx name="hokuyo1" parent="base_link">
+		<origin xyz="-0.1 0.0 0.33" rpy="0 0 0"/>
+	</xacro:sensor_hokuyo_urg04lx>
 -->
-  <xacro:sensor_axis name="camera" parent="base_link">
+	<xacro:sensor_axis name="camera" parent="base_link">
 		<origin xyz="0.19 0 0.17" rpy="0 ${15*PI/180} 0"/>
-  </xacro:sensor_axis>
-  <xacro:sensor_imu name="imu" parent="base_link">
+	</xacro:sensor_axis>
+	<xacro:sensor_imu name="imu" parent="base_link">
 		<origin xyz="-0.18 0.0 0.170" rpy="0 0 0"/>
-  </xacro:sensor_imu>
-  <xacro:sensor_gps name="gps" parent="base_link">
+	</xacro:sensor_imu>
+	<xacro:sensor_gps name="gps" parent="base_link">
 		<origin xyz="-0.22 0 0.275" rpy="0 0 0"/>
 	</xacro:sensor_gps>
 <!--
-  <xacro:sensor_kinect name="kinect" parent="base_link">
-    <origin xyz="0.3 0.0 0.16" rpy="0 0 0"/>
-  </xacro:sensor_kinect>
+	<xacro:sensor_kinect name="kinect" parent="base_link">
+		<origin xyz="0.3 0.0 0.16" rpy="0 0 0"/>
+	</xacro:sensor_kinect>
 -->
 <!--
-  <xacro:sensor_fotonic name="fotonic" parent="base_link">
-    <origin xyz="0.3 0.0 0.24" rpy="0 0 0"/>
-  </xacro:sensor_fotonic>
+	<xacro:sensor_fotonic name="fotonic" parent="base_link">
+		<origin xyz="0.3 0.0 0.24" rpy="0 0 0"/>
+	</xacro:sensor_fotonic>
 -->
 </robot>

Commit message: summit_xl_description: unifying the rubber wheels in only one .dae file

File: summit_xl_description/robots/summit_xl.urdf.xacro (robot description, xacro)
@@ -32,14 +32,14 @@
 	<xacro:skid_steering/>
 	<!-- WHEELS -->
-	<xacro:rubber_wheel name="front_right" parent="base_link" reflect="0" hq="${hq}">
+	<xacro:rubber_wheel name="front_right" parent="base_link" reflect="false" hq="${hq}">
 		<origin xyz="${wheel_offset_x} -${wheel_offset_y} ${wheel_offset_z}" rpy="0 0 0"/>
 	</xacro:rubber_wheel>
-	<xacro:rubber_wheel name="front_left" parent="base_link" reflect="1" hq="${hq}">
+	<xacro:rubber_wheel name="front_left" parent="base_link" reflect="true" hq="${hq}">
 		<origin xyz="${wheel_offset_x} ${wheel_offset_y} ${wheel_offset_z}" rpy="0 0 0"/>
 	</xacro:rubber_wheel>
-	<xacro:rubber_wheel name="back_left" parent="base_link" reflect="1" hq="${hq}">
+	<xacro:rubber_wheel name="back_left" parent="base_link" reflect="true" hq="${hq}">
 		<origin xyz="-${wheel_offset_x} ${wheel_offset_y} ${wheel_offset_z}" rpy="0 0 0"/>
 	</xacro:rubber_wheel>
-	<xacro:rubber_wheel name="back_right" parent="base_link" reflect="0" hq="${hq}">
+	<xacro:rubber_wheel name="back_right" parent="base_link" reflect="false" hq="${hq}">
 		<origin xyz="-${wheel_offset_x} -${wheel_offset_y} ${wheel_offset_z}" rpy="0 0 0"/>
 	</xacro:rubber_wheel>

File: summit_xl_description/urdf/bases/summit_xl_base.gazebo.xacro (robot description, xacro)
@@ -48,14 +48,3 @@
     <material>Gazebo/Green</material>
   </gazebo>
-<!--
-  <gazebo reference="base_link">
-    <material>Gazebo/Black</material>
-  </gazebo>
-  <gazebo reference="logos_link">
-    <material>Gazebo/Red</material>
-  </gazebo>
-  <gazebo reference="covers_link">
-    <material>Gazebo/Grey</material>
-  </gazebo>
--->
 </robot>

File: summit_xl_description/urdf/wheels/rubber_wheel.urdf.xacro (robot description, xacro)
@@ -27,5 +27,10 @@
           <origin xyz="0 0 0" rpy="0 0 0" />
           <geometry>
-            <mesh filename="package://summit_xl_description/meshes/wheels/rubber_wheel.dae" />
+						<xacro:if value="${reflect}">
+							<mesh filename="package://summit_xl_description/meshes/wheels/rubber_wheel_left.dae" />
+						</xacro:if>
+						<xacro:unless value="${reflect}">
+							<mesh filename="package://summit_xl_description/meshes/wheels/rubber_wheel_right.dae" />
+						</xacro:unless>
           </geometry>
         </xacro:if>
@@ -37,12 +42,7 @@
           </geometry>
         </xacro:unless>
-<!--
-        <material name="darkgrey">
-           <color rgba="0.2 0.2 0.2 1"/>
-        </material>
--->
       </visual>
       <collision>
-		<origin xyz="0 0 0" rpy="${M_PI/2} 0 0" />
+				<origin xyz="0 0 0" rpy="${M_PI/2} 0 0" />
         <geometry>
           <cylinder length="${wheel_height}" radius="${wheel_radius}" />
@@ -55,32 +55,4 @@
       </inertial>
     </link>
-<!-- WHEEL COVERS -->
-    <joint name="joint_cover_${name}_wheel" type="fixed">
-      <parent link="${name}_wheel"/>
-      <child link="cover_${name}1_wheel"/>
-      <origin xyz="0 0 0" rpy="0 0 0"/>
-    </joint>
-     <link name="cover_${name}1_wheel">
-      <visual>
-		<origin xyz="0 0 0" rpy="${reflect*PI} 0 0" />
-        <geometry>
-          <mesh filename="package://summit_xl_description/meshes/wheels/rubber_wheel_cover.dae" />
-        </geometry>
-<!--
-        <material name="lightgrey">
-           <color rgba="0.6 0.6 0.6 1"/>
-        </material>
--->
-      </visual>
-<!-- MOTOR VISUAL -->
-<!--
-      <visual>
-        <origin xyz="0 0 0" rpy="${M_PI/2} 0 0" />
-        <geometry>
-          <cylinder length="${wheel_height}" radius="0.05" />
-        </geometry>
-      </visual>
--->
-     </link>
     <!-- Transmission is important to link the joints and the controller (see summit_xl_control/config/summit_xl_control.yaml)-->
     <transmission name="${name}_wheel_joint_trans">
@@ -98,9 +70,5 @@
 			<kd value="1.0" />
 			<fdir1 value="1 0 0"/>
-			<material>Gazebo/Black</material>
       <turnGravityOff>false</turnGravityOff>
-    </gazebo>
-    <gazebo reference="cover_${name}1_wheel">
-      <material>Gazebo/Grey</material>
     </gazebo>
   </xacro:macro>

Commit message: Asus Xtion Pro description added.

File: summit_xl_description/robots/summit_xl.urdf.xacro (robot description, xacro)
@@ -63,4 +63,9 @@
 	</xacro:sensor_gps>
 <!--
+	<xacro:sensor_asus_xtion_pro name="xtion_pro" parent="base_link">
+		<origin xyz="0.3 0.0 0.3" rpy="0 0 0"/>
+	</xacro:sensor_asus_xtion_pro>
+-->
+<!--
 	<xacro:sensor_kinect name="kinect" parent="base_link">
 		<origin xyz="0.3 0.0 0.16" rpy="0 0 0"/>

File: summit_xl_description/urdf/sensors/all_sensors.urdf.xacro (robot description, xacro)
@@ -16,3 +16,5 @@
   <!-- Kinect -->
   <xacro:include filename="$(find summit_xl_description)/urdf/sensors/kinect.urdf.xacro" />
+  <!-- Asus Xtion PRO -->
+  <xacro:include filename="$(find summit_xl_description)/urdf/sensors/asus_xtion_pro.urdf.xacro" />
 </robot>
