Commit message: ros_control plugin removed from .gazebo.xacro to allow modular robot assemblies

File: summit_xl_description/robots/summit_xl_standalone.urdf.xacro (robot description, xacro)
@@ -11,4 +11,12 @@
 	<!-- Import all available sensors -->
 	<xacro:include filename="$(find summit_xl_description)/urdf/sensors/all_sensors.urdf.xacro" />
+    <gazebo>
+      <plugin name="ros_control" filename="libgazebo_ros_control.so">
+        <robotNamespace>/summit_xl</robotNamespace>
+        <robotParam>robot_description</robotParam>
+        <controlPeriod>0.001</controlPeriod>
+	    <robotSimType>gazebo_ros_control/DefaultRobotHWSim</robotSimType>
+      </plugin>
+    </gazebo>
 	<!-- ***************** -->
 	<!-- Global parameters -->

File: summit_xl_description/urdf/bases/summit_xl_base.gazebo.xacro (robot description, xacro)
@@ -2,5 +2,5 @@
 <robot xmlns:xacro="http://ros.org/wiki/xacro">
   <!-- ros control plugin -->
-  <xacro:macro name="ros_control">
+  <!-- xacro:macro name="ros_control">
     <gazebo>
       <plugin name="ros_control" filename="libgazebo_ros_control.so">
@@ -11,5 +11,5 @@
       </plugin>
     </gazebo>
-	</xacro:macro>
+	</xacro:macro -->
 	<!-- skid steering plugin -->
 	<xacro:macro name="skid_steering" params="broadcastOdomTF">
