Commit message: summit_xl_description: adding IMU sensor to Summit X robot

File: summit_xl_description/robots/summit_x.urdf.xacro (robot description, xacro)
@@ -26,4 +26,5 @@
 	<!-- Here we create the robot elements using the xacro:macros imported at the beggining of this file -->
 	<!-- Summit XL base -->
+	<!-- this base already includes the Axis camera and Hokuyo laser sensors -->
 	<xacro:summit_x_base name="summit_xl" publish_bf="true" />
 	<!-- Gazebo ros control pluggins -->
@@ -64,9 +65,7 @@
 	</xacro:sensor_axis>
 -->
-<!--
-	<xacro:sensor_imu name="imu" parent="base_link">
-		<origin xyz="-0.18 0.0 0.170" rpy="0 0 0"/>
+	<xacro:sensor_imu name="imu" parent="rover_link">
+		<origin xyz="-0.30 0.0 0.1" rpy="0 0 0"/>
 	</xacro:sensor_imu>
--->
 <!--
 	<xacro:sensor_gps name="gps" parent="base_link">

Commit message: summit_xl_description: adding xacro parameter to broadcast odom TF

File: summit_xl_description/robots/summit_x.urdf.xacro (robot description, xacro)
@@ -32,5 +32,5 @@
 	<!-- Gazebo skid steering pluggins -->
 <!--
-	<xacro:skid_steering/>
+	<xacro:skid_steering broadcastOdomTF="0"/>
 -->
 	<!-- Gazebo omni steering plugin -->

File: summit_xl_description/robots/summit_xl.urdf.xacro (robot description, xacro)
@@ -30,5 +30,5 @@
 	<xacro:ros_control/>
 	<!-- Gazebo skid steering pluggins -->
-	<xacro:skid_steering/>
+	<xacro:skid_steering broadcastOdomTF="0"/>
 	<!-- WHEELS -->
 	<xacro:rubber_wheel name="front_right" parent="base_link" reflect="false" hq="${hq}">

File: summit_xl_description/urdf/bases/summit_x_base.gazebo.xacro (robot description, xacro)
@@ -13,5 +13,5 @@
 	</xacro:macro>
 	<!-- skid steering plugin -->
-	<xacro:macro name="skid_steering">
+	<xacro:macro name="skid_steering" params="broadcastOdomTF">
     <gazebo>
       <plugin name="skid_steer_drive_controller" filename="libgazebo_ros_skid_steer_drive.so">
@@ -30,5 +30,5 @@
 	    <odometryTopic>odom</odometryTopic>
 	    <odometryFrame>/odom</odometryFrame>
-	    <broadcastTF>true</broadcastTF>
+	    <broadcastTF>${broadcastOdomTF}</broadcastTF>
       </plugin>
     </gazebo>

File: summit_xl_description/urdf/bases/summit_xl_base.gazebo.xacro (robot description, xacro)
@@ -13,5 +13,5 @@
 	</xacro:macro>
 	<!-- skid steering plugin -->
-	<xacro:macro name="skid_steering">
+	<xacro:macro name="skid_steering" params="broadcastOdomTF">
     <gazebo>
       <plugin name="skid_steer_drive_controller" filename="libgazebo_ros_skid_steer_drive.so">
@@ -30,5 +30,5 @@
 		    <odometryTopic>odom</odometryTopic>
 		    <odometryFrame>/odom</odometryFrame>
-		    <broadcastTF>1</broadcastTF>
+		    <broadcastTF>${broadcastOdomTF}</broadcastTF>
       </plugin>
     </gazebo>

Commit message: summit_xl_description: fixing kinect sensor frames

File: summit_xl_description/robots/summit_x.urdf.xacro (robot description, xacro)
@@ -75,5 +75,5 @@
 <!--
 	<xacro:sensor_kinect name="kinect" parent="base_link">
-		<origin xyz="0.3 0.0 0.16" rpy="0 0 0"/>
+		<origin xyz="0.325 0.0 0.16" rpy="0 0 0"/>
 	</xacro:sensor_kinect>
 -->

File: summit_xl_description/robots/summit_xl.urdf.xacro (robot description, xacro)
@@ -69,5 +69,5 @@
 <!--
 	<xacro:sensor_kinect name="kinect" parent="base_link">
-		<origin xyz="0.3 0.0 0.16" rpy="0 0 0"/>
+		<origin xyz="0.325 0.0 0.16" rpy="0 0 0"/>
 	</xacro:sensor_kinect>
 -->

File: summit_xl_description/robots/summit_xl_nocam.urdf.xacro (robot description, xacro)
@@ -71,5 +71,5 @@
 <!--
 	<xacro:sensor_kinect name="kinect" parent="base_link">
-		<origin xyz="0.3 0.0 0.16" rpy="0 0 0"/>
+		<origin xyz="0.325 0.0 0.16" rpy="0 0 0"/>
 	</xacro:sensor_kinect>
 -->

File: summit_xl_description/robots/summit_xl_omni.urdf.xacro (robot description, xacro)
@@ -64,5 +64,5 @@
 <!--
 	<xacro:sensor_kinect name="kinect" parent="base_link">
-		<origin xyz="0.3 0.0 0.16" rpy="0 0 0"/>
+		<origin xyz="0.325 0.0 0.16" rpy="0 0 0"/>
 	</xacro:sensor_kinect>
 -->

File: summit_xl_description/robots/summit_xl_standalone.urdf.xacro (robot description, xacro)
@@ -75,9 +75,7 @@
 	</xacro:sensor_asus_xtion_pro>
 -->
-<!--
 	<xacro:sensor_kinect name="kinect" parent="base_link">
-		<origin xyz="0.3 0.0 0.16" rpy="0 0 0"/>
+		<origin xyz="0.325 0.0 0.16" rpy="0 0 0"/>
 	</xacro:sensor_kinect>
--->
 <!--
 	<xacro:sensor_fotonic name="fotonic" parent="base_link">

File: summit_xl_description/urdf/sensors/kinect.urdf.xacro (robot description, xacro)
@@ -2,37 +2,17 @@
 <robot name="sensor_kinect" xmlns:xacro="http://ros.org/wiki/xacro">
   <xacro:property name="M_PI" value="3.1415926535897931" />
+	<xacro:property name="cam_px" value="-0.087" />
+	<xacro:property name="cam_py" value="-0.0125" />
+	<xacro:property name="cam_pz" value="0.2870" />
+	<xacro:property name="cam_or" value="0" />
+	<xacro:property name="cam_op" value="0" />
+	<xacro:property name="cam_oy" value="0" />
   <xacro:macro name="sensor_kinect" params="name parent *origin">
-    <joint name="${name}_cam_joint" type="fixed">
-	    <insert_block name="origin" />
-	    <parent link="${parent}"/>
-	    <child link="${name}_cam_link"/>
-	  </joint>
-	  <link name="${name}_cam_link">
-	    <visual>
-	     <origin xyz="0 0 0" rpy="0 0 ${M_PI/2}"/>
-	      <geometry>
-	       <mesh filename="package://summit_xl_description/meshes/sensors/kinect.dae"/>
-	      </geometry>
-	    </visual>
-		  <collision>
-	      <origin xyz="0.0 0.0 0.0" rpy="0 0 0"/>
-		    <geometry>
-		      <box size="0.07271 0.27794 0.073"/>
-		    </geometry>
-		  </collision>
-	    <inertial>
-	      <mass value="0.001" />
-	      <origin xyz="0 0 0" />
-	      <inertia ixx="0.0001" ixy="0.0" ixz="0.0"
-	               iyy="0.0001" iyz="0.0"
-	               izz="0.0001" />
-	    </inertial>
-	  </link>
-    <joint name="${name}_cam_rgb_joint" type="fixed">
-      <origin xyz="0.031 -0.0125 0.016" rpy="0 0 0"/>
-      <parent link="${name}_cam_link"/>
-      <child link="${name}_cam_rgb_frame" />
+    <joint name="${name}_rgb_joint" type="fixed">
+      <insert_block name="origin" />
+      <parent link="${parent}"/>
+      <child link="${name}_rgb_frame" />
     </joint>
-    <link name="${name}_cam_rgb_frame">
+    <link name="${name}_rgb_frame">
       <inertial>
         <mass value="0.001" />
@@ -43,10 +23,10 @@
       </inertial>
     </link>
-    <joint name="${name}_cam_rgb_optical_joint" type="fixed">
+    <joint name="${name}_rgb_optical_joint" type="fixed">
       <origin xyz="0 0 0" rpy="${-M_PI/2} 0 ${-M_PI/2}" />
-      <parent link="${name}_cam_rgb_frame" />
-      <child link="${name}_cam_rgb_optical_frame" />
+      <parent link="${name}_rgb_frame" />
+      <child link="${name}_rgb_optical_frame" />
     </joint>
-    <link name="${name}_cam_rgb_optical_frame">
+    <link name="${name}_rgb_optical_frame">
       <inertial>
         <mass value="0.001" />
@@ -57,40 +37,66 @@
       </inertial>
     </link>
-	  <!-- The fixed joints & links below are usually published by static_transformers launched by the OpenNi launch
-	       files. However, for Gazebo simulation we need them, so we add them here.
-	       (Hence, don't publish them additionally!) -->
-		<joint name="${name}_cam_depth_joint" type="fixed">
-		  <origin xyz="0 0.025 0" rpy="0 0 0" />
-		  <parent link="${name}_cam_rgb_frame" />
-		  <child link="${name}_cam_depth_frame" />
-		</joint>
-		<link name="${name}_cam_depth_frame">
-	    <inertial>
-	      <mass value="0.001" />
-	      <origin xyz="0 0 0" />
-	      <inertia ixx="0.0001" ixy="0.0" ixz="0.0"
-	               iyy="0.0001" iyz="0.0"
-	               izz="0.0001" />
-	    </inertial>
-		</link>
-		<joint name="${name}_cam_depth_optical_joint" type="fixed">
-		  <origin xyz="0 0 0" rpy="${-M_PI/2} 0 ${-M_PI/2}" />
-		  <parent link="${name}_cam_depth_frame" />
-		  <child link="${name}_cam_depth_optical_frame" />
-		</joint>
-		<link name="${name}_cam_depth_optical_frame">
-	    <inertial>
-	      <mass value="0.001" />
-	      <origin xyz="0 0 0" />
-	      <inertia ixx="0.0001" ixy="0.0" ixz="0.0"
-	               iyy="0.0001" iyz="0.0"
-	               izz="0.0001" />
-	    </inertial>
-		</link>
+  <joint name="${name}_joint" type="fixed">
+    <origin xyz="-0.031 ${-cam_py} -0.016" rpy="0 0 0"/>
+    <parent link="${name}_rgb_frame"/>
+    <child link="${name}_link"/>
+  </joint>
+    <link name="${name}_link">
+    <visual>
+     <origin xyz="0 0 0" rpy="0 0 ${M_PI/2}"/>
+      <geometry>
+       <mesh filename="package://summit_xl_description/meshes/sensors/kinect.dae"/>
+      </geometry>
+    </visual>
+	  <collision>
+      <origin xyz="0.0 0.0 0.0" rpy="0 0 0"/>
+	    <geometry>
+	      <box size="0.07271 0.27794 0.073"/>
+	    </geometry>
+	  </collision>
+    <inertial>
+      <mass value="0.001" />
+      <origin xyz="0 0 0" />
+      <inertia ixx="0.0001" ixy="0.0" ixz="0.0"
+               iyy="0.0001" iyz="0.0"
+               izz="0.0001" />
+    </inertial>
+  </link>
+  <!-- The fixed joints & links below are usually published by static_transformers launched by the OpenNi launch
+       files. However, for Gazebo simulation we need them, so we add them here.
+       (Hence, don't publish them additionally!) -->
+	<joint name="${name}_depth_joint" type="fixed">
+	  <origin xyz="0 ${2 * -cam_py} 0" rpy="0 0 0" />
+	  <parent link="${name}_rgb_frame" />
+	  <child link="${name}_depth_frame" />
+	</joint>
+	<link name="${name}_depth_frame">
+    <inertial>
+      <mass value="0.001" />
+      <origin xyz="0 0 0" />
+      <inertia ixx="0.0001" ixy="0.0" ixz="0.0"
+               iyy="0.0001" iyz="0.0"
+               izz="0.0001" />
+    </inertial>
+	</link>
+	<joint name="${name}_depth_optical_joint" type="fixed">
+	  <origin xyz="0 0 0" rpy="${-M_PI/2} 0 ${-M_PI/2}" />
+	  <parent link="${name}_depth_frame" />
+	  <child link="${name}_depth_optical_frame" />
+	</joint>
+	<link name="${name}_depth_optical_frame">
+    <inertial>
+      <mass value="0.001" />
+      <origin xyz="0 0 0" />
+      <inertia ixx="0.0001" ixy="0.0" ixz="0.0"
+               iyy="0.0001" iyz="0.0"
+               izz="0.0001" />
+    </inertial>
+	</link>
 		<!-- Kinect sensor for simulation -->
 	  <sensor_kinect_gazebo/>
   </xacro:macro>
   <xacro:macro name="sensor_kinect_gazebo">
-    <gazebo reference="${name}_cam_depth_frame">
+    <gazebo reference="${name}_link">
       <sensor type="depth" name="cam">
         <always_on>true</always_on>
@@ -117,5 +123,5 @@
           <cameraInfoTopicName>rgb/camera_info</cameraInfoTopicName>
           <depthImageCameraInfoTopicName>depth/camera_info</depthImageCameraInfoTopicName>
-          <frameName>${name}_cam_depth_optical_frame</frameName>
+          <frameName>${name}_depth_optical_frame</frameName>
           <baseline>0.1</baseline>
           <distortion_k1>0.0</distortion_k1>
